File: Composite Designs/C30 Pocket Controller/Eagle/Skaarhoj BI8-SE-C30.brd (EAGLE design)
At the start: 73.7 x 72.4 mm, 54 parts, among them IC1 MCP23017SS, IC2 PCA9685, U1 ARDUINO_SHIELDNO_SILK

Commit message: Numerous updates to PCBs including a whole new design, C330 (in the making)
Parts:
- R1, R2: value 10K -> 1K5
Changed lines of the file:
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@@
 </autorouter>
 <elements>
-<element name="R1" library="SparkFun" package="0603-RES" value="10K" x="26.2255" y="16.256" smashed="yes" rot="MR180">
+<element name="R1" library="SparkFun" package="0603-RES" value="1K5" x="26.2255" y="16.256" smashed="yes" rot="MR180">
 <attribute name="NAME" x="23.8125" y="15.494" size="0.8128" layer="26" font="vector" rot="MR180"/>
 <attribute name="VALUE" x="25.2095" y="17.399" size="0.4064" layer="28" font="vector" rot="MR180"/>
 </element>
-<element name="R2" library="SparkFun" package="0603-RES" value="10K" x="26.2255" y="14.0335" smashed="yes" rot="MR180">
+<element name="R2" library="SparkFun" package="0603-RES" value="1K5" x="26.2255" y="14.0335" smashed="yes" rot="MR180">
 <attribute name="NAME" x="23.9395" y="13.2715" size="0.8128" layer="26" font="vector" rot="MR180"/>
 <attribute name="VALUE" x="25.2095" y="15.1765" size="0.4064" layer="28" font="vector" rot="MR180"/>
@@
 </signal>
 </signals>
-<errors>
-</errors>
 </board>
 </drawing>
