File: PCB Design/BI8 series boards/Skaarhoj BI8-1x8CAP3slim.brd (EAGLE design)
At the start: 147.3 x 29 mm, 45 parts, among them IC1 MCP23017SS, IC2 PCA9685

Commit message: Various updated and new stuff
Parts:
- removed R1, R2: 10K, SparkFun:0603-RES
- removed RN1: 10K, SKAARHOJ:CAY16_HAND
- removed S1: SWS002, smd-special:SMS-002
- added SJ6, SJ7, SJ8: SOLDERJUMPERNC, SparkFun:SJ_2S
- moved SJ5 6.99 mm to (135.9, 22.9)
- moved SJ3 3.59 mm to (135.9, 26.7)
- moved SJ4 3.18 mm to (135.9, 24.8)
Connections:
- net 5VL: no longer R1.1, R2.1, S1.1, S1.2
- net A0: now also SJ6.2; no longer RN1.5, S1.4
- net A1: now also SJ7.2; no longer RN1.6, S1.3
- net A2: now also SJ8.2; no longer RN1.7
- net GNDL: now also SJ6.1, SJ7.1, SJ8.1; no longer RN1.1, RN1.2, RN1.3, RN1.4
- net I2C_SCL: no longer R2.2
- net I2C_SDA: no longer R1.2
Routing:
- net 5VL: track 119.7 -> 94.8 mm, vias 7 -> 6
- net I2C_SCL: track 78.0 -> 57.3 mm
- net A1: track 95.9 -> 112.3 mm, vias 2 -> 3
- net I2C_SDA: track 75.0 -> 64.7 mm
- net A0: track 75.5 -> 82.2 mm, vias 2 -> 8
- net GNDL: track 182.6 -> 187.9 mm, vias 4 -> 5
- net A2: track 73.9 -> 71.4 mm, vias 4 -> 5
- net GND: vias 2 -> 3
Other:
- board text added: ""0""
- board text added: ""1""
- board text added: "A0"
- board text added: "A1"
- board text added: "v26-03-13"
- board text removed: "I2C Pullups"
- board text removed: "v03-01-13"
