File: PCBs/PCB-BI8-SE-C330/PCB-BI8-SE-C330.sch (EAGLE design)
At the start: 36 parts, among them IC1 MCP23017SS, IC2 PCA9685

Commit message: Large revisions of boards, change of forms, in particular all mounting holes now has a 7mm diameter and fully inside the board.
Parts:
- removed R1, R2: 10K, SparkFun:RESISTOR0603-RES
- removed RN1: 10K, SKAARHOJ:4R-NCAY16
- removed S1: SWS003, smd-special:SWS003
- removed SJ1, SJ2: SOLDERJUMPERNC, SparkFun:SOLDERJUMPERNC
- added U$15, U$18, U$20, U$21: GNDPAD6MM, SKAARHOJ:GNDPAD6MM
- added U$19: 3BITADDR, SKAARHOJ:3BITADDR
Connections:
- removed net 5VL: IC1.!RESET, IC2.A3, IC2.A4, IC2.A5, R1.1, R2.1, S1.4, S1.5, S1.6, SJ1.2
- removed net GNDL: B1.SW1, B2.SW1, B3.SW1, B4.SW1, B5.SW1, B6.SW1, B7.SW1, B8.SW1, IC1.GPB0, IC2.EXTCLK, IC2.OE, RN1A.1, RN1B.1, RN1C.1, RN1D.1, SJ2.2
- net 5V: now also IC2.A3, IC2.A4, IC2.A5, U$19.VCC; no longer SJ1.1
- net A0: now also U$19.A0; no longer RN1D.2, S1.3
- net A1: now also U$19.A1; no longer RN1C.2, S1.2
- net A2: now also U$19.A2; no longer RN1B.2, S1.1
- net GND: now also B1.SW1, B2.SW1, B3.SW1, B4.SW1, B5.SW1, B6.SW1, B7.SW1, B8.SW1, IC1.!RESET, IC1.GPB0, IC2.EXTCLK, IC2.OE, U$15.1, U$18.1, U$19.GND, U$20.1, U$21.1; no longer SJ2.1
- net I2C_SCL: no longer R2.2
- net I2C_SDA: no longer R1.2
