File: PCBs/PCB-ACMb/PCB-ACMb.brd (EAGLE design)
At the start: 59.7 x 35.6 mm, 59 parts, among them IC1 MCP23017SS, IC2 PCA9685

Commit message: new and updated PCBs. Schaeffer Housing script
Parts:
- LED1, LED10, LED11, LED12, LED13, LED14, LED15, LED16, LED2, LED3, LED4, LED5, LED6, LED7, LED8, LED9: value (none) -> LED3MM; device SparkFun:LED3MM -> SKAARHOJ:LED3MM
- moved LED10 0.25 mm to (9.00, 24.0)
- moved LED11 0.25 mm to (13.0, 24.0)
- moved LED12 0.25 mm to (17.0, 24.0)
- moved LED13 0.25 mm to (21.0, 24.0)
- moved LED14 0.25 mm to (25.0, 24.0)
- moved LED15 0.25 mm to (29.0, 24.0)
- moved LED9 0.25 mm to (5.00, 24.0)
- moved LED16 0.25 mm to (33.0, 24.0)
- moved LED2 0.23 mm to (9.00, 31.0)
- moved LED3 0.23 mm to (13.0, 31.0)
- moved LED1 0.23 mm to (5.00, 31.0)
- moved LED4 0.23 mm to (17.0, 31.0)
- moved LED5 0.23 mm to (21.0, 31.0)
- moved LED6 0.23 mm to (25.0, 31.0)
- moved LED7 0.23 mm to (29.0, 31.0)
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Routing:
- net 5V: track 213.9 -> 218.9 mm
