File: PCBs/PCB-CMB-5-SHLD/PCB-CMB-5-SHLD__testWDisp.sch (EAGLE design)
At the start: 87 parts, among them IC1 ULN2803A, IC2 MCP23017SS, IC3 PCA9685, IC4 MCP23017SS, K1 RELAY5VIM03, K2 RELAY5VIM03, K3 RELAY5VIM03, K4 RELAY5VIM03, K5 RELAY5VIM03, K6 RELAY5VIM03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

Commit message: asdf
Parts:
- added U1: (no value), SKAARHOJ:ER-OLED0.91-2
- R29: device SparkFun:RESISTOR0603-RES -> SparkFun:RESISTOR1206
Changed lines of the file:
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@@
 <layer number="106" name="bPlate" color="7" fill="1" visible="yes" active="yes"/>
 <layer number="107" name="Crop" color="7" fill="1" visible="yes" active="yes"/>
+<layer number="108" name="tBridges" color="7" fill="1" visible="yes" active="yes"/>
+<layer number="109" name="tBPL" color="7" fill="1" visible="yes" active="yes"/>
+<layer number="110" name="bBPL" color="7" fill="1" visible="yes" active="yes"/>
+<layer number="111" name="MPL" color="7" fill="1" visible="yes" active="yes"/>
+<layer number="112" name="tSilk" color="7" fill="1" visible="yes" active="yes"/>
 <layer number="116" name="Patch_BOT" color="9" fill="4" visible="no" active="yes"/>
 <layer number="121" name="_tsilk" color="7" fill="1" visible="yes" active="yes"/>
@@
 <layer number="125" name="_tNames" color="7" fill="1" visible="yes" active="yes"/>
 <layer number="126" name="_bNames" color="7" fill="1" visible="yes" active="yes"/>
+<layer number="127" name="_tValues" color="7" fill="1" visible="yes" active="yes"/>
+<layer number="128" name="_bValues" color="7" fill="1" visible="yes" active="yes"/>
 <layer number="144" name="Drill_legend" color="7" fill="1" visible="no" active="yes"/>
 <layer number="151" name="HeatSink" color="7" fill="1" visible="no" active="yes"/>
+<layer number="152" name="_bDocu" color="7" fill="1" visible="yes" active="yes"/>
 <layer number="199" name="L$199" color="7" fill="1" visible="yes" active="yes"/>
 <layer number="200" name="200bmp" color="1" fill="10" visible="no" active="yes"/>
@@
 <layer number="223" name="223bmp" color="24" fill="1" visible="no" active="no"/>
 <layer number="224" name="224bmp" color="25" fill="1" visible="no" active="no"/>
+<layer number="248" name="Housing" color="7" fill="1" visible="yes" active="yes"/>
+<layer number="249" name="Edge" color="7" fill="1" visible="yes" active="yes"/>
 <layer number="250" name="Descript" color="3" fill="1" visible="no" active="no"/>
 <layer number="251" name="SMDround" color="12" fill="11" visible="no" active="no"/>
@@
 <part name="R27" library="SparkFun" deviceset="RESISTOR" device="0603-RES" value="100R"/>
 <part name="R28" library="SparkFun" deviceset="RESISTOR" device="0603-RES" value="100R"/>
-<part name="R29" library="SparkFun" deviceset="RESISTOR" device="0603-RES" value="100R"/>
+<part name="R29" library="SparkFun" deviceset="RESISTOR" device="1206" value="100R"/>
 <part name="R30" library="SparkFun" deviceset="RESISTOR" device="0603-RES" value="100R"/>
 <part name="R31" library="SparkFun" deviceset="RESISTOR" device="0603-RES" value="100R"/>
@@
 <part name="U$3" library="SparkFun" deviceset="5V" device=""/>
 <part name="U$4" library="SKAARHOJ" deviceset="GNDPAD" device="6MM" value="GNDPAD6MM"/>
+<part name="U1" library="SKAARHOJ" deviceset="ER-OLED0.91-2" device=""/>
 </parts>
 <sheets>
@@
 <instance part="U$3" gate="G$1" x="101.6" y="205.74"/>
 <instance part="U$4" gate="G$1" x="231.14" y="213.36"/>
+<instance part="U1" gate="G$1" x="-165.1" y="203.2"/>
 </instances>
 <busses>
