File: PCBs/PCB-ARD-DUEBOS/PCB-ARD-DUEBOS.sch (EAGLE design)
At the start: 55 parts, among them IC2 MCP3008SOIC, IC3 MCP3008SOIC, Q1 BSS138, Q2 BSS138, U1 ARDUINO-MEGAFULL, U2 74HC4050D, U3 74HC4050D, U4 74HC4050D, U5 74HC4050D, U6 74HC4050D

Commit message: Various changes
Parts:
- removed C7: 0.1uF, SparkFun:CAP0603-CAP
- removed JP8: (no value), SparkFun:M02PTH4
- removed U$35: M24C64, SKAARHOJ:M24C64
- added C8: 0.1uF, SparkFun:CAP0603-CAP
- added U7: (no value), microbuilder:EEPROM_SPI_AT25040ATSSOP
- added X1, X2: MSTBV23.5MM, SKAARHOJ:MSTBV23.5MM
- Q1, Q2: device microbuilder:MOSFET-NWIDE -> microbuilder:MOSFET-NREFLOW
- R1, R2, R3, R4: value 10K -> 1K5; device microbuilder:RESISTOR0805 -> microbuilder:RESISTOR0603
Connections:
- removed net EEPROM_WC: U$35._WC, U1.44
- removed net N$25: U1.46
- removed net N$26: U1.45
- new net EEPROM_CS: U1.44, U7.CS
- net 3.3V: now also C8.1, U7.HOLD, U7.VCC, U7.WP; no longer C7.1, U$35.E0, U$35.E1, U$35.E2, U$35.VCC
- net 5V: now also X1-2.1; no longer JP8.2
- net GND: now also C8.2, U7.GND, X1-1.1, X2-1.1; no longer C7.2, JP8.1, U$35.VSS
- net MISO_3.3V: now also U7.MISO
- net MOSI_3.3V: now also U7.MOSI
- net SCLK_3.3V: now also U7.SCK
- net SCL_3.3V: no longer U$35.SCL
- net SDA_3.3V: no longer U$35.SDA
- net VIN: now also X2-2.1
Other:
- note added: "POWER IN/OUTLET"
- note removed: "POWER OUTLET"
