File: PCBs/PCB-BI8-3x5C3/PCB-BI8-3x5C3_V2.brd (EAGLE design)
At the start: 86.4 x 94 mm, 71 parts, among them IC1 MCP23017SS, IC2 PCA9685, IC3 PCA9685

Commit message: asdf
Parts:
- added B1ALT, B2ALT, B3ALT, B4ALT: LP11-B", SKAARHOJ:LP11
- moved C2 52.2 mm to (34.2, 54.9)
- moved IC2 51.8 mm to (27.9, 54.6)
- moved R11 4.74 mm to (76.1, 17.3), turned to 0 degrees
- moved R15 4.74 mm to (40.5, 17.3), turned to 0 degrees
- moved R12 4.74 mm to (76.1, 13.2), turned to 0 degrees
- moved R16 4.74 mm to (40.5, 13.2), turned to 0 degrees
- moved R20 4.74 mm to (4.95, 13.2), turned to 0 degrees
- moved R14 4.74 mm to (58.3, 13.2), turned to 0 degrees
- moved R18 4.74 mm to (22.7, 13.2), turned to 0 degrees
- moved R19 4.74 mm to (4.95, 17.3), turned to 0 degrees
- moved R13 4.74 mm to (58.3, 17.3), turned to 0 degrees
- moved R17 4.74 mm to (22.7, 17.3), turned to 0 degrees
- moved IC1 2.54 mm to (14.7, 55.0)
- moved C1 1.97 mm to (8.51, 54.9)
- turned B1 to 180 degrees
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Connections:
- net 5V: now also B1ALT.COM, B2ALT.COM, B3ALT.COM, B4ALT.COM
- net GND: now also B1ALT.P$4, B2ALT.P$4, B3ALT.P$4, B4ALT.P$4
- net GPA4: now also B1ALT.P$5
- net GPA5: now also B2ALT.P$5
- net GPA6: now also B3ALT.P$5
- net GPA7: now also B4ALT.P$5
- net L0: now also B1ALT.P$2
- net L1: now also B1ALT.P$3
- net L2: now also B2ALT.P$2
- net L3: now also B2ALT.P$3
- net L4: now also B3ALT.P$2
- net L5: now also B3ALT.P$3
- net L6: now also B4ALT.P$2
- net L7: now also B4ALT.P$3
Routing:
- added copper zone on layer 1, net GND
- added copper zone on layer 16, net GND
