File: PCBs/PCB-BI8-3x5C3/PCB-BI8-3x5C3_V2.sch (EAGLE design)
At the start: 41 parts, among them IC1 MCP23017SS, IC2 PCA9685

Commit message: asdf
Parts:
- removed B5ALT: LP11-B", SKAARHOJ:LP11-B"
- removed U$22, U$23: GNDPAD6MM, SKAARHOJ:GNDPAD6MM
- added B10, B10ALT, B11, B11ALT, B12, B12ALT, B13, B13ALT, B14, B14ALT, B15, B15ALT, B16, B2ALT, B3ALT, B9, B9ALT: LP11-B", SKAARHOJ:LP11-B"
- added C5: 100nF, SparkFun:CAP0603-CAP
- added IC3: PCA9685, wsmith:PCA9685
- added R1, R2, R21, R22, R23, R24, R25, R26, R27, R28, R29, R3, R30, R31, R32, R4: 270, SparkFun:RESISTOR0603-RES
- added U$15, U$18: GNDPAD6MM, SKAARHOJ:GNDPAD6MM
- R5: SEEEDOPL asdf -> (none)
Connections:
- new net GPA10: B14.SW2, B14ALT.SW2, IC1.GPB2
- new net GPA11: B13.SW2, B13ALT.SW2, IC1.GPB3
- new net GPA12: B9.SW2, B9ALT.SW2, IC1.GPB4
- new net GPA13: B10.SW2, B10ALT.SW2, IC1.GPB5
- new net GPA14: B11.SW2, B11ALT.SW2, IC1.GPB6
- new net GPA15: B12.SW2, B12ALT.SW2, IC1.GPB7
- new net GPA8: B16.SW2, IC1.GPB0
- new net GPA9: B15.SW2, B15ALT.SW2, IC1.GPB1
- new net L16: B9.K1, B9ALT.K1, R32.1
- new net L17: B9.K2, B9ALT.K2, R31.1
- new net L18: B10.K1, B10ALT.K1, R30.1
- new net L19: B10.K2, B10ALT.K2, R29.1
- new net L20: B11.K1, B11ALT.K1, R28.1
- new net L21: B11.K2, B11ALT.K2, R27.1
- new net L22: B12.K1, B12ALT.K1, R26.1
- new net L23: B12.K2, B12ALT.K2, R25.1
- new net L24: B13.K1, B13ALT.K1, R24.1
- new net L25: B13.K2, B13ALT.K2, R23.1
- new net L26: B14.K1, B14ALT.K1, R22.1
- new net L27: B14.K2, B14ALT.K2, R21.1
- new net L28: B15.K1, B15ALT.K1, R4.1
- new net L29: B15.K2, B15ALT.K2, R3.1
- new net L30: B16.K1, R2.1
- new net L31: B16.K2, R1.1
- new net N$1: IC3.L7, R25.2
- new net N$13: IC3.L2, R30.2
- new net N$14: IC3.L1, R31.2
- new net N$15: IC3.L0, R32.2
- new net N$16: IC3.L8, R24.2
- new net N$17: IC3.L9, R23.2
- new net N$18: IC3.L10, R22.2
- new net N$2: IC3.L6, R26.2
- new net N$28: IC3.L11, R21.2
- new net N$29: IC3.L12, R4.2
- new net N$3: IC3.L5, R27.2
- new net N$30: IC3.L13, R3.2
- new net N$31: IC3.L14, R2.2
- new net N$32: IC3.L15, R1.2
- new net N$6: IC3.L4, R28.2
- new net N$8: IC3.L3, R29.2
- net 5V: now also B10.A, B10ALT.A, B11.A, B11ALT.A, B12.A, B12ALT.A, B13.A, B13ALT.A, B14.A, B14ALT.A, B15.A, B15ALT.A, B16.A, B2ALT.A, B3ALT.A, B9.A, B9ALT.A, C5.1, IC3.A5, IC3.VDD; no longer B5ALT.A
- net A0: now also IC3.A0
- net A1: now also IC3.A1
- net A2: now also IC3.A2
- net GND: now also B10.SW1, B10ALT.SW1, B11.SW1, B11ALT.SW1, B12.SW1, B12ALT.SW1, B13.SW1, B13ALT.SW1, B14.SW1, B14ALT.SW1, B15.SW1, B15ALT.SW1, B16.SW1, B2ALT.SW1, B3ALT.SW1, B9.SW1, B9ALT.SW1, C5.2, IC3.A3, IC3.A4, IC3.EXTCLK, IC3.GND, IC3.OE, U$15.1, U$18.1; no longer B5ALT.SW1, IC1.GPB0, U$22.1, U$23.1
- net GPA3: no longer B5ALT.SW2
- net GPA5: now also B2ALT.SW2
- net GPA6: now also B3ALT.SW2
- net I2C_SCL: now also IC3.SCL
- net I2C_SDA: now also IC3.SDA
- net L2: now also B2ALT.K1
- net L3: now also B2ALT.K2
- net L4: now also B3ALT.K1
- net L5: now also B3ALT.K2
- net L8: no longer B5ALT.K1
- net L9: no longer B5ALT.K2
Other:
- note added: "ADR=B100xxx"
