File: PCBs/PCB-BI8-3x5C3/PCB-BI8-3x5C3.sch (EAGLE design)
At the start: 67 parts, among them IC1 MCP23017SS, IC2 PCA9685, IC3 PCA9685

Commit message: asdf
Parts:
- removed B16ALT, B1ALT, B4ALT: LP11-B", SKAARHOJ:LP11-B"
- added B10ALT, B11ALT, B12ALT, B14ALT, B15ALT, B6ALT, B7ALT: LP11-B", SKAARHOJ:LP11-B"
Connections:
- net 5V: now also B10ALT.A, B11ALT.A, B12ALT.A, B14ALT.A, B15ALT.A, B6ALT.A, B7ALT.A; no longer B16ALT.A, B1ALT.A, B4ALT.A
- net GND: now also B10ALT.SW1, B11ALT.SW1, B12ALT.SW1, B14ALT.SW1, B15ALT.SW1, B6ALT.SW1, B7ALT.SW1; no longer B16ALT.SW1, B1ALT.SW1, B4ALT.SW1
- net GPA1: now also B7ALT.SW2
- net GPA10: now also B14ALT.SW2
- net GPA13: now also B10ALT.SW2
- net GPA14: now also B11ALT.SW2
- net GPA15: now also B12ALT.SW2
- net GPA2: now also B6ALT.SW2
- net GPA4: no longer B1ALT.SW2
- net GPA7: no longer B4ALT.SW2
- net GPA8: no longer B16ALT.SW2
- net GPA9: now also B15ALT.SW2
- net L0: no longer B1ALT.K1
- net L1: no longer B1ALT.K2
- net L10: now also B6ALT.K1
- net L11: now also B6ALT.K2
- net L12: now also B7ALT.K1
- net L13: now also B7ALT.K2
- net L18: now also B10ALT.K1
- net L19: now also B10ALT.K2
- net L20: now also B11ALT.K1
- net L21: now also B11ALT.K2
- net L22: now also B12ALT.K1
- net L23: now also B12ALT.K2
- net L26: now also B14ALT.K1
- net L27: now also B14ALT.K2
- net L28: now also B15ALT.K1
- net L29: now also B15ALT.K2
- net L30: no longer B16ALT.K1
- net L31: no longer B16ALT.K2
- net L6: no longer B4ALT.K1
- net L7: no longer B4ALT.K2
Other:
- moved on the sheet: B1, B10, B11, B12, B13, B13ALT, B14, B15, B16, B2, B3, B4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

Commit message: PCBS updated
Parts:
- removed B16: LP11-B", SKAARHOJ:LP11-B"
- removed C3: 10uF, SparkFun:CAP0805
- removed R1, R2: 270, SparkFun:RESISTOR0603-RES
- added C10, C6, C7, C8, C9: 100nF, SparkFun:CAP0603-CAP
- added C4: 22uF, SparkFun:CAP0805
- added L4: ILHB0805ER121V, SparkFun:INDUCTOR0805
Connections:
- removed net L30: B16.K1, R2.1
- removed net L31: B16.K2, R1.1
- removed net N$31: IC3.L14, R2.2
- removed net N$32: IC3.L15, R1.2
- new net N$33: C7.1, L4.1, SERIAL.2
- net 5V: now also C10.1, C4.1, C6.1, C8.1, C9.1, L4.2; no longer B16.A, C3.1, SERIAL.2
- net GND: now also C10.2, C4.2, C6.2, C7.2, C8.2, C9.2; no longer B16.SW1, C3.2
- net GPA8: no longer B16.SW2
Other:
- note removed: "POWER"
