File: PCBs/PCB-DISPARRAY4b/PCB-DISPARRAY4b.sch (EAGLE design)
At the start: 51 parts, among them U1 74HC4050D, U3 74HC4050D, U5 FAN5331SX

Commit message: Various changes
Parts:
- removed U$10, U$9: GNDPAD6MM, SKAARHOJ:GNDPAD6MM
- C15, C20, C25, C6: device SparkFun:CAP0603-CAP -> SparkFun:CAP0805
- C19: device microbuilder:CAP_CERAMIC0805 -> microbuilder:CAP_CERAMIC0603
- R6, R7: device microbuilder:RESISTOR0805 -> microbuilder:RESISTOR0603
- U1, U3: device microbuilder:74HC4050D -> SKAARHOJ:74HC4050DTSSOP16
- U4, U6, U7, U8: device SKAARHOJ:ER-OLED011-1 -> SKAARHOJ:ER-OLED011-1TOP
Connections:
- new net DPWR_3V3: U1.6Y, U5.SHDN
- new net DPWR_5V: U$23.P15, U1.6A
- net 3.3V: no longer U5.SHDN
- net 5V: no longer U$19.VCC
- net GND: no longer U$10.1, U$19.GND, U$9.1, U1.6A
- net I2C_SCL: now also U$19.VCC
- net I2C_SDA: now also U$19.GND

Commit message: a lot
Parts:
- added C27: 10uF/25V, SparkFun:CAP0805
- R6: value 50K -> 51K
Connections:
- net 7.5V: now also C27.2
- net GND: now also C27.1
Other:
- note added: "7.5V Boost"
- note added: "VOUT = 7.5V"
- note removed: "13V Boost"
- note removed: "VOUT = 13.53V"
Changed lines of the file:
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@@
 <part name="L1" library="microbuilder" deviceset="INDUCTOR" device="" value="10uH"/>
 <part name="D3" library="microbuilder" deviceset="DIODE" device="SOD-123" value="BAT54T1G"/>
-<part name="R6" library="microbuilder" deviceset="RESISTOR" device="0603" value="50K"/>
+<part name="R6" library="microbuilder" deviceset="RESISTOR" device="0603" value="51K"/>
 <part name="R7" library="microbuilder" deviceset="RESISTOR" device="0603" value="10K"/>
 <part name="U$3" library="microbuilder" deviceset="GND" device=""/>
@@
 <part name="C25" library="SparkFun" deviceset="CAP" device="0805" value="10uF"/>
 <part name="C26" library="SparkFun" deviceset="CAP" device="0603-CAP" value="100nF"/>
+<part name="C27" library="SparkFun" deviceset="CAP" device="0805" value="10uF/25V"/>
 </parts>
 <sheets>
@@
 <text x="-182.88" y="25.4" size="1.778" layer="91">Based on schematics from Adafruit! Thanks!</text>
 <text x="127" y="-185.42" size="1.778" layer="97">VOUT = 1.23V * (1 + R6/R7)</text>
-<text x="127" y="-187.96" size="1.778" layer="97">VOUT = 13.53V</text>
+<text x="127" y="-187.96" size="1.778" layer="97">VOUT = 7.5V</text>
 <text x="111.76" y="-193.04" size="1.778" layer="97">This is 0.5V above the recommended voltage,</text>
 <text x="111.76" y="-195.58" size="1.778" layer="97">but uses common resistors for easy assembly</text>
-<text x="137.16" y="-134.62" size="1.778" layer="97">13V Boost</text>
+<text x="137.16" y="-134.62" size="1.778" layer="97">7.5V Boost</text>
 <text x="114.3" y="-203.2" size="1.778" layer="91">Booster circuit from Adafruit, thanks!</text>
 <text x="-182.88" y="-76.2" size="1.778" layer="91">Based on schematics from Adafruit! Thanks!</text>
@@
 <instance part="C25" gate="G$1" x="-124.46" y="-292.1" rot="R180"/>
 <instance part="C26" gate="G$1" x="-111.76" y="-292.1" rot="R180"/>
+<instance part="C27" gate="G$1" x="185.42" y="-160.02" rot="R180"/>
 </instances>
 <busses>
@@
 <pinref part="R7" gate="G$1" pin="1"/>
 <pinref part="U$3" gate="G$1" pin="GND"/>
+<pinref part="C27" gate="G$1" pin="1"/>
+<wire x1="185.42" y1="-165.1" x2="185.42" y2="-175.26" width="0.1524" layer="91"/>
+<wire x1="185.42" y1="-175.26" x2="167.64" y2="-175.26" width="0.1524" layer="91"/>
+<junction x="167.64" y="-175.26"/>
 </segment>
 <segment>
@@
 <pinref part="7.5V1" gate="1" pin="VCC"/>
 <junction x="175.26" y="-142.24"/>
-</segment>
-<segment>
+<pinref part="C27" gate="G$1" pin="2"/>
+<wire x1="175.26" y1="-142.24" x2="185.42" y2="-142.24" width="0.1524" layer="91"/>
+<wire x1="185.42" y1="-142.24" x2="185.42" y2="-157.48" width="0.1524" layer="91"/>
+</segment>
+<segment>

Commit message: asdf
Parts:
- renumbered U4 to DISP1, U6 to DISP2, U7 to DISP3, U8 to DISP4

Commit message: PCBS updated
Connections:
- net I2C_SCL: now also U$19.GND; no longer U$19.VCC
- net I2C_SDA: now also U$19.VCC; no longer U$19.GND
Changed lines of the file:
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@@
 </segment>
 <segment>
-<pinref part="U$19" gate="G$1" pin="GND"/>
-<wire x1="142.24" y1="-17.78" x2="144.78" y2="-17.78" width="0.1524" layer="91"/>
-<label x="144.78" y="-17.78" size="1.778" layer="95"/>
+<pinref part="U$19" gate="G$1" pin="VCC"/>
+<wire x1="142.24" y1="-15.24" x2="144.78" y2="-15.24" width="0.1524" layer="91"/>
+<label x="144.78" y="-15.24" size="1.778" layer="95"/>
 </segment>
 </net>
@@
 </segment>
 <segment>
-<pinref part="U$19" gate="G$1" pin="VCC"/>
-<wire x1="142.24" y1="-15.24" x2="144.78" y2="-15.24" width="0.1524" layer="91"/>
-<label x="144.78" y="-15.24" size="1.778" layer="95"/>
+<pinref part="U$19" gate="G$1" pin="GND"/>
+<wire x1="142.24" y1="-17.78" x2="144.78" y2="-17.78" width="0.1524" layer="91"/>
+<label x="144.78" y="-17.78" size="1.778" layer="95"/>
 </segment>
 </net>
