File: PCBs/PCB-TLY-JACK-MEGA/PCB-TLY-JACK-MEGA.brd (EAGLE design)
At the start: 159.4 x 73.7 mm, 102 parts, among them IC1 ULN2803A, IC2 MCP23017SS, K1 RELAY5VIM03, K2 RELAY5VIM03, K3 RELAY5VIM03, K4 RELAY5VIM03, K5 RELAY5VIM03, K6 RELAY5VIM03, K7 RELAY5VIM03, K8 RELAY5VIM03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

Commit message: PCBS updated
Parts:
- U$11: value Tally 1-2-3 -> PRG Tally 1-2-3
- U$12: value Tally 2-3-4 -> PRG Tally 4-5-6
- U$13: value Tally 3-4-1 -> PRG Tally 7-8
Changed lines of the file:
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@@
 <?xml version="1.0" encoding="utf-8"?>
 <!DOCTYPE eagle SYSTEM "eagle.dtd">
-<eagle version="6.5.0">
+<eagle version="7.1.0">
 <drawing>
 <settings>
@@
 <pass name="Default">
 <param name="RoutingGrid" value="4mil"/>
+<param name="AutoGrid" value="1"/>
+<param name="Efforts" value="0"/>
+<param name="TopRouterVariant" value="1"/>
 <param name="tpViaShape" value="round"/>
 <param name="PrefDir.1" value="-"/>
@@
 <element name="LED32" library="led" package="LED3MM" value="" x="57.5" y="22" rot="R270"/>
 <element name="LED33" library="led" package="LED3MM" value="" x="57.5" y="16"/>
-<element name="U$11" library="SKAARHOJ" package="RJ45-8_GND_UPRIGHT" value="Tally 1-2-3" x="26" y="14"/>
-<element name="U$12" library="SKAARHOJ" package="RJ45-8_GND_UPRIGHT" value="Tally 2-3-4" x="47" y="14"/>
-<element name="U$13" library="SKAARHOJ" package="RJ45-8_GND_UPRIGHT" value="Tally 3-4-1" x="68" y="14"/>
+<element name="U$11" library="SKAARHOJ" package="RJ45-8_GND_UPRIGHT" value="PRG Tally 1-2-3" x="26" y="14"/>
+<element name="U$12" library="SKAARHOJ" package="RJ45-8_GND_UPRIGHT" value="PRG Tally 4-5-6" x="47" y="14"/>
+<element name="U$13" library="SKAARHOJ" package="RJ45-8_GND_UPRIGHT" value="PRG Tally 7-8" x="68" y="14"/>
 <element name="RN3" library="SKAARHOJ" package="RN-9" value="" x="91.5" y="31.5" rot="MR180">
 <attribute name="OC_NEWARK" value="unknown" x="91.5" y="31.5" size="1.778" layer="28" rot="MR180" display="off"/>
