File: PCBs/PCB-REMCON-ER/PCB-REMCON-ER.sch (EAGLE design)
At the start: 11 parts

Commit message: asfd
Parts:
- removed JOY1: M04X2, SparkFun:M04X2
- removed R6, R7: 100R, SparkFun:RESISTOR0603-RES
- removed SCLK->D1, SCLK->D5: SOLDERJUMPERNC, SparkFun:SOLDERJUMPERNC
- removed Z1, Z2: 5V1, SparkFun:DIODE-ZENERSMB
Connections:
- removed net N$1: R6.2, SERIAL.3
- removed net N$14: R7.1, SERIAL.4
- removed net POT1: JOY1.2, SCLK->D1.2, U$2.5
- removed net POT2: JOY1.3, SCLK->D5.2, U$2.6
- net 5V: now also U$2.5, U$2.7; no longer JOY1.7, U$2.2
- net GND: now also U$2.3; no longer JOY1.8, Z1.A, Z2.A
- net I2C_SCL: now also SERIAL.4; no longer R7.2, Z2.C
- net I2C_SDA: now also SERIAL.3, U$2.8; no longer R6.1, U$2.3, Z1.C
- net N$4: no longer SCLK->D5.1
- net N$5: no longer SCLK->D1.1
- net SDI_MOSI: now also U$2.2; no longer U$2.8
- net SDI_SCLK: now also U$2.6; no longer U$2.7
Other:
- note removed: "JOYSTICK"
