File: PCBs/PCB-CARR-SL45/PCB-CARR-SL45.sch (EAGLE design)
At the start: 3 parts

Commit message: PCB updates
Parts:
- added POT2: SLIDERC45, SKAARHOJ:SLIDERC45
Connections:
- net 5V: now also POT2.E
- net ANALOG1: now also POT2.S
- net GND: now also POT2.A
Other:
- note removed: "CHANNEL"
