File: PCBs/PCB-ENCODER4/PCB-ENCODER4.sch (EAGLE design)
At the start: 37 parts, among them IC1 MCP23017SS, IC2 74HC14D, SW1 EC12E_SW, SW2 EC12E_SW, SW3 EC12E_SW, SW4 EC12E_SW

Commit message: PCBS updated
Parts:
- C1: value 10uF -> 22uF
- C11, C2, C5, C8: value 100nF -> 10nF
- R1, R3, R4, R5, R6: value 10K -> 100K
- R13, R2, R22, R31, R7: value 10K -> 0R
Changed lines of the file:
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@@
 <part name="GND1" library="SparkFun" deviceset="GND" device=""/>
 <part name="SW1" library="switch-alps" deviceset="EC12E_SW" device=""/>
-<part name="C1" library="SparkFun" deviceset="CAP" device="0805" value="10uF"/>
-<part name="C2" library="SparkFun" deviceset="CAP" device="0603-CAP" value="100nF"/>
+<part name="C1" library="SparkFun" deviceset="CAP" device="0805" value="22uF"/>
+<part name="C2" library="SparkFun" deviceset="CAP" device="0603-CAP" value="10nF"/>
 <part name="C3" library="SparkFun" deviceset="CAP" device="0603-CAP" value="10nF"/>
 <part name="C4" library="SparkFun" deviceset="CAP" device="0603-CAP" value="10nF"/>
 <part name="U$2" library="SparkFun" deviceset="5V" device=""/>
 <part name="GND2" library="SparkFun" deviceset="GND" device=""/>
-<part name="R2" library="SparkFun" deviceset="RESISTOR" device="0603-RES" value="10K"/>
+<part name="R2" library="SparkFun" deviceset="RESISTOR" device="0603-RES" value="0R"/>
 <part name="U$20" library="SKAARHOJ" deviceset="GNDPAD" device="6MM" value="GNDPAD6MM"/>
 <part name="U$21" library="SKAARHOJ" deviceset="GNDPAD" device="6MM" value="GNDPAD6MM"/>
@@
 <part name="GND3" library="SparkFun" deviceset="GND" device=""/>
 <part name="SW2" library="switch-alps" deviceset="EC12E_SW" device=""/>
-<part name="C5" library="SparkFun" deviceset="CAP" device="0603-CAP" value="100nF"/>
+<part name="C5" library="SparkFun" deviceset="CAP" device="0603-CAP" value="10nF"/>
 <part name="C6" library="SparkFun" deviceset="CAP" device="0603-CAP" value="10nF"/>
 <part name="C7" library="SparkFun" deviceset="CAP" device="0603-CAP" value="10nF"/>
-<part name="R13" library="SparkFun" deviceset="RESISTOR" device="0603-RES" value="10K"/>
+<part name="R13" library="SparkFun" deviceset="RESISTOR" device="0603-RES" value="0R"/>
 <part name="GND4" library="SparkFun" deviceset="GND" device=""/>
 <part name="SW3" library="switch-alps" deviceset="EC12E_SW" device=""/>
-<part name="C8" library="SparkFun" deviceset="CAP" device="0603-CAP" value="100nF"/>
+<part name="C8" library="SparkFun" deviceset="CAP" device="0603-CAP" value="10nF"/>
 <part name="C9" library="SparkFun" deviceset="CAP" device="0603-CAP" value="10nF"/>
 <part name="C10" library="SparkFun" deviceset="CAP" device="0603-CAP" value="10nF"/>
-<part name="R22" library="SparkFun" deviceset="RESISTOR" device="0603-RES" value="10K"/>
+<part name="R22" library="SparkFun" deviceset="RESISTOR" device="0603-RES" value="0R"/>
 <part name="GND5" library="SparkFun" deviceset="GND" device=""/>
 <part name="SW4" library="switch-alps" deviceset="EC12E_SW" device=""/>
-<part name="C11" library="SparkFun" deviceset="CAP" device="0603-CAP" value="100nF"/>
+<part name="C11" library="SparkFun" deviceset="CAP" device="0603-CAP" value="10nF"/>
 <part name="C12" library="SparkFun" deviceset="CAP" device="0603-CAP" value="10nF"/>
 <part name="C13" library="SparkFun" deviceset="CAP" device="0603-CAP" value="10nF"/>
-<part name="R31" library="SparkFun" deviceset="RESISTOR" device="0603-RES" value="10K"/>
+<part name="R31" library="SparkFun" deviceset="RESISTOR" device="0603-RES" value="0R"/>
 <part name="IC1" library="microchip" deviceset="MCP23017" device="SS">
 <attribute name="MPN" value="MCP23017-E/SS"/>
@@
 <part name="U$1" library="SKAARHOJ" deviceset="M02X2" device=""/>
 <part name="IC2" library="74xx-eu" deviceset="74*14" device="D" technology="HC"/>
-<part name="R6" library="SparkFun" deviceset="RESISTOR" device="0603-RES" value="10K"/>
+<part name="R6" library="SparkFun" deviceset="RESISTOR" device="0603-RES" value="100K"/>
 <part name="U$7" library="SparkFun" deviceset="5V" device=""/>
 <part name="GND9" library="SparkFun" deviceset="GND" device=""/>
 <part name="U$9" library="SparkFun" deviceset="5V" device=""/>
 <part name="C18" library="SparkFun" deviceset="CAP" device="0603-CAP" value="100nF"/>
-<part name="R1" library="SparkFun" deviceset="RESISTOR" device="0603-RES" value="10K"/>
-<part name="R3" library="SparkFun" deviceset="RESISTOR" device="0603-RES" value="10K"/>
-<part name="R4" library="SparkFun" deviceset="RESISTOR" device="0603-RES" value="10K"/>
-<part name="R5" library="SparkFun" deviceset="RESISTOR" device="0603-RES" value="10K"/>
+<part name="R1" library="SparkFun" deviceset="RESISTOR" device="0603-RES" value="100K"/>
+<part name="R3" library="SparkFun" deviceset="RESISTOR" device="0603-RES" value="100K"/>
+<part name="R4" library="SparkFun" deviceset="RESISTOR" device="0603-RES" value="100K"/>
+<part name="R5" library="SparkFun" deviceset="RESISTOR" device="0603-RES" value="100K"/>
 <part name="U$3" library="SparkFun" deviceset="5V" device=""/>
 <part name="U$4" library="SparkFun" deviceset="5V" device=""/>
 <part name="U$5" library="SparkFun" deviceset="5V" device=""/>
 <part name="U$6" library="SparkFun" deviceset="5V" device=""/>
-<part name="R7" library="SparkFun" deviceset="RESISTOR" device="0603-RES" value="10K"/>
+<part name="R7" library="SparkFun" deviceset="RESISTOR" device="0603-RES" value="0R"/>
 </parts>
 <sheets>

Commit message: asdf
Parts:
- removed R13, R2, R22, R31, R7: 0R, SparkFun:RESISTOR0603-RES
Connections:
- removed net N$1: R2.2, R3.1, SW1G$1.B
- removed net N$12: R31.2, R5.1, SW4G$1.B
- removed net N$127: R6.1, R7.1, U$1.2
- removed net N$6: R13.2, R4.1, SW2G$1.B
- removed net N$9: R1.1, R22.2, SW3G$1.B
- net N$123: now also R1.1, SW3G$1.B; no longer R22.1
- net N$124: now also R3.1, SW1G$1.B; no longer R2.1
- net N$125: now also R4.1, SW2G$1.B; no longer R13.1
- net N$126: now also R5.1, SW4G$1.B; no longer R31.1
- net N$2: now also R6.1, U$1.2; no longer R7.2
Changed lines of the file:
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@@
 <?xml version="1.0" encoding="utf-8"?>
 <!DOCTYPE eagle SYSTEM "eagle.dtd">
-<eagle version="7.1.0">
+<eagle version="7.2.0">
 <drawing>
 <settings>
@@
 <part name="U$2" library="SparkFun" deviceset="5V" device=""/>
 <part name="GND2" library="SparkFun" deviceset="GND" device=""/>
-<part name="R2" library="SparkFun" deviceset="RESISTOR" device="0603-RES" value="0R"/>
 <part name="U$20" library="SKAARHOJ" deviceset="GNDPAD" device="6MM" value="GNDPAD6MM"/>
 <part name="U$21" library="SKAARHOJ" deviceset="GNDPAD" device="6MM" value="GNDPAD6MM"/>
@@
 <part name="C6" library="SparkFun" deviceset="CAP" device="0603-CAP" value="10nF"/>
 <part name="C7" library="SparkFun" deviceset="CAP" device="0603-CAP" value="10nF"/>
-<part name="R13" library="SparkFun" deviceset="RESISTOR" device="0603-RES" value="0R"/>
 <part name="GND4" library="SparkFun" deviceset="GND" device=""/>
 <part name="SW3" library="switch-alps" deviceset="EC12E_SW" device=""/>
@@
 <part name="C9" library="SparkFun" deviceset="CAP" device="0603-CAP" value="10nF"/>
 <part name="C10" library="SparkFun" deviceset="CAP" device="0603-CAP" value="10nF"/>
-<part name="R22" library="SparkFun" deviceset="RESISTOR" device="0603-RES" value="0R"/>
 <part name="GND5" library="SparkFun" deviceset="GND" device=""/>
 <part name="SW4" library="switch-alps" deviceset="EC12E_SW" device=""/>
@@
 <part name="C12" library="SparkFun" deviceset="CAP" device="0603-CAP" value="10nF"/>
 <part name="C13" library="SparkFun" deviceset="CAP" device="0603-CAP" value="10nF"/>
-<part name="R31" library="SparkFun" deviceset="RESISTOR" device="0603-RES" value="0R"/>
 <part name="IC1" library="microchip" deviceset="MCP23017" device="SS">
 <attribute name="MPN" value="MCP23017-E/SS"/>
@@
 <part name="U$5" library="SparkFun" deviceset="5V" device=""/>
 <part name="U$6" library="SparkFun" deviceset="5V" device=""/>
-<part name="R7" library="SparkFun" deviceset="RESISTOR" device="0603-RES" value="0R"/>
 </parts>
 <sheets>
@@
 <instance part="U$2" gate="G$1" x="162.56" y="104.14"/>
 <instance part="GND2" gate="1" x="162.56" y="93.98"/>
-<instance part="R2" gate="G$1" x="-53.34" y="144.78"/>
 <instance part="U$20" gate="G$1" x="147.32" y="73.66"/>
 <instance part="U$21" gate="G$1" x="175.26" y="73.66"/>
@@
 <instance part="C6" gate="G$1" x="27.94" y="111.76"/>
 <instance part="C7" gate="G$1" x="17.78" y="111.76"/>
-<instance part="R13" gate="G$1" x="50.8" y="144.78"/>
 <instance part="GND4" gate="1" x="-66.04" y="35.56"/>
 <instance part="SW3" gate="G$1" x="-12.7" y="76.2" rot="R90"/>
@@
 <instance part="C9" gate="G$1" x="-76.2" y="45.72"/>
 <instance part="C10" gate="G$1" x="-86.36" y="45.72"/>
-<instance part="R22" gate="G$1" x="-53.34" y="78.74"/>
 <instance part="GND5" gate="1" x="38.1" y="35.56"/>
 <instance part="SW4" gate="G$1" x="91.44" y="76.2" rot="R90"/>
@@
 <instance part="C12" gate="G$1" x="27.94" y="45.72"/>
 <instance part="C13" gate="G$1" x="17.78" y="45.72"/>
-<instance part="R31" gate="G$1" x="50.8" y="78.74"/>
 <instance part="IC1" gate="G$1" x="-167.64" y="124.46" rot="R180"/>
 <instance part="U$13" gate="G$1" x="-142.24" y="104.14"/>
@@
 <instance part="U$6" gate="G$1" x="-43.18" y="88.9"/>
 <instance part="IC2" gate="B" x="17.78" y="-27.94" rot="R180"/>
-<instance part="R7" gate="G$1" x="48.26" y="10.16" rot="R180"/>
 </instances>
 <busses>
@@
 </segment>
 </net>
-<net name="N$1" class="0">
-<segment>
-<pinref part="SW1" gate="G$1" pin="B"/>
-<pinref part="R2" gate="G$1" pin="2"/>
-<wire x1="-48.26" y1="144.78" x2="-43.18" y2="144.78" width="0.1524" layer="91"/>
-<pinref part="R3" gate="G$1" pin="1"/>
-<wire x1="-43.18" y1="144.78" x2="-20.32" y2="144.78" width="0.1524" layer="91"/>
-<junction x="-43.18" y="144.78"/>
-</segment>
-</net>
 <net name="I2C_SDA" class="0">
 <segment>
@@
 </segment>
 </net>
-<net name="N$6" class="0">
-<segment>
-<pinref part="SW2" gate="G$1" pin="B"/>
-<pinref part="R13" gate="G$1" pin="2"/>
-<wire x1="55.88" y1="144.78" x2="60.96" y2="144.78" width="0.1524" layer="91"/>
-<pinref part="R4" gate="G$1" pin="1"/>
-<wire x1="60.96" y1="144.78" x2="83.82" y2="144.78" width="0.1524" layer="91"/>
-<junction x="60.96" y="144.78"/>
-</segment>
-</net>
-<net name="N$9" class="0">
-<segment>
-<pinref part="SW3" gate="G$1" pin="B"/>
-<pinref part="R22" gate="G$1" pin="2"/>
-<wire x1="-48.26" y1="78.74" x2="-43.18" y2="78.74" width="0.1524" layer="91"/>
-<pinref part="R1" gate="G$1" pin="1"/>
-<wire x1="-43.18" y1="78.74" x2="-20.32" y2="78.74" width="0.1524" layer="91"/>
-<junction x="-43.18" y="78.74"/>
-</segment>
-</net>
-<net name="N$12" class="0">
-<segment>
-<pinref part="SW4" gate="G$1" pin="B"/>
-<pinref part="R31" gate="G$1" pin="2"/>
-<wire x1="55.88" y1="78.74" x2="60.96" y2="78.74" width="0.1524" layer="91"/>
-<pinref part="R5" gate="G$1" pin="1"/>
-<wire x1="60.96" y1="78.74" x2="83.82" y2="78.74" width="0.1524" layer="91"/>
-<junction x="60.96" y="78.74"/>
-</segment>
-</net>
 <net name="A0" class="0">
 <segment>
@@
 <wire x1="-66.04" y1="50.8" x2="-66.04" y2="78.74" width="0.1524" layer="91"/>
 <wire x1="-66.04" y1="78.74" x2="-58.42" y2="78.74" width="0.1524" layer="91"/>
-<pinref part="R22" gate="G$1" pin="1"/>
 <junction x="-66.04" y="78.74"/>
 <wire x1="-78.74" y1="81.28" x2="-73.66" y2="81.28" width="0.1524" layer="91"/>
@@
 <wire x1="-73.66" y1="78.74" x2="-66.04" y2="78.74" width="0.1524" layer="91"/>
 <pinref part="IC2" gate="F" pin="I"/>
+<pinref part="SW3" gate="G$1" pin="B"/>
+<wire x1="-48.26" y1="78.74" x2="-43.18" y2="78.74" width="0.1524" layer="91"/>
+<pinref part="R1" gate="G$1" pin="1"/>
+<wire x1="-43.18" y1="78.74" x2="-20.32" y2="78.74" width="0.1524" layer="91"/>
+<junction x="-43.18" y="78.74"/>
+<wire x1="-66.04" y1="78.74" x2="-43.18" y2="78.74" width="0.1524" layer="91"/>
 </segment>
 </net>
@@
 <wire x1="-66.04" y1="116.84" x2="-66.04" y2="144.78" width="0.1524" layer="91"/>
 <wire x1="-66.04" y1="144.78" x2="-58.42" y2="144.78" width="0.1524" layer="91"/>
-<pinref part="R2" gate="G$1" pin="1"/>
 <junction x="-66.04" y="144.78"/>
 <pinref part="IC2" gate="A" pin="I"/>
 <wire x1="-78.74" y1="144.78" x2="-66.04" y2="144.78" width="0.1524" layer="91"/>
+<pinref part="SW1" gate="G$1" pin="B"/>
+<wire x1="-48.26" y1="144.78" x2="-43.18" y2="144.78" width="0.1524" layer="91"/>
+<pinref part="R3" gate="G$1" pin="1"/>
+<wire x1="-43.18" y1="144.78" x2="-20.32" y2="144.78" width="0.1524" layer="91"/>
+<junction x="-43.18" y="144.78"/>
+<wire x1="-66.04" y1="144.78" x2="-43.18" y2="144.78" width="0.1524" layer="91"/>
 </segment>
 </net>
@@
 <wire x1="38.1" y1="116.84" x2="38.1" y2="144.78" width="0.1524" layer="91"/>
 <wire x1="38.1" y1="144.78" x2="45.72" y2="144.78" width="0.1524" layer="91"/>
-<pinref part="R13" gate="G$1" pin="1"/>
 <junction x="38.1" y="144.78"/>
 <pinref part="IC2" gate="C" pin="I"/>
 <wire x1="27.94" y1="144.78" x2="38.1" y2="144.78" width="0.1524" layer="91"/>
+<pinref part="SW2" gate="G$1" pin="B"/>
+<wire x1="55.88" y1="144.78" x2="60.96" y2="144.78" width="0.1524" layer="91"/>
+<pinref part="R4" gate="G$1" pin="1"/>
+<wire x1="60.96" y1="144.78" x2="83.82" y2="144.78" width="0.1524" layer="91"/>
+<junction x="60.96" y="144.78"/>
+<wire x1="38.1" y1="144.78" x2="60.96" y2="144.78" width="0.1524" layer="91"/>
 </segment>
 </net>
@@
 <wire x1="38.1" y1="50.8" x2="38.1" y2="78.74" width="0.1524" layer="91"/>
 <wire x1="38.1" y1="78.74" x2="45.72" y2="78.74" width="0.1524" layer="91"/>
-<pinref part="R31" gate="G$1" pin="1"/>
 <junction x="38.1" y="78.74"/>
 <pinref part="IC2" gate="E" pin="I"/>
 <wire x1="38.1" y1="78.74" x2="27.94" y2="78.74" width="0.1524" layer="91"/>
-</segment>
-</net>
-<net name="N$127" class="0">
-<segment>
+<pinref part="SW4" gate="G$1" pin="B"/>
+<wire x1="55.88" y1="78.74" x2="60.96" y2="78.74" width="0.1524" layer="91"/>
+<pinref part="R5" gate="G$1" pin="1"/>
+<wire x1="60.96" y1="78.74" x2="83.82" y2="78.74" width="0.1524" layer="91"/>
+<junction x="60.96" y="78.74"/>
+<wire x1="38.1" y1="78.74" x2="60.96" y2="78.74" width="0.1524" layer="91"/>
+</segment>
+</net>
+<net name="N$2" class="0">
+<segment>
+<pinref part="IC2" gate="D" pin="I"/>
+<wire x1="43.18" y1="10.16" x2="27.94" y2="10.16" width="0.1524" layer="91"/>
 <pinref part="R6" gate="G$1" pin="1"/>
 <pinref part="U$1" gate="G$1" pin="2"/>
@@
 <wire x1="93.98" y1="0" x2="93.98" y2="10.16" width="0.1524" layer="91"/>
 <wire x1="93.98" y1="10.16" x2="71.12" y2="10.16" width="0.1524" layer="91"/>
-<pinref part="R7" gate="G$1" pin="1"/>
 <wire x1="53.34" y1="10.16" x2="71.12" y2="10.16" width="0.1524" layer="91"/>
 <junction x="71.12" y="10.16"/>
-</segment>
-</net>
-<net name="N$2" class="0">
-<segment>
-<pinref part="R7" gate="G$1" pin="2"/>
-<pinref part="IC2" gate="D" pin="I"/>
-<wire x1="43.18" y1="10.16" x2="27.94" y2="10.16" width="0.1524" layer="91"/>
-</segment>
-</net>
+<wire x1="27.94" y1="10.16" x2="71.12" y2="10.16" width="0.1524" layer="91"/>
+<junction x="27.94" y="10.16"/>
+</segment>
+</net>

Commit message: PCB updates
Parts:
- SERIAL: value M04X2 -> M04X2M2X4SMALLER; device SparkFun:M04X2 -> SKAARHOJ:M04X2M2X4SMALLER
- U$19: value 3BITADDR -> 3BITADDRSMALL; device SKAARHOJ:3BITADDR -> SKAARHOJ:3BITADDRSMALL
Changed lines of the file:
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@@
 <?xml version="1.0" encoding="utf-8"?>
 <!DOCTYPE eagle SYSTEM "eagle.dtd">
-<eagle version="7.2.0">
+<eagle version="7.5.0">
 <drawing>
 <settings>
@@
 <layer number="56" name="wert" color="7" fill="1" visible="no" active="no"/>
 <layer number="57" name="tCAD" color="7" fill="1" visible="no" active="no"/>
+<layer number="90" name="Modules" color="5" fill="1" visible="yes" active="yes"/>
 <layer number="91" name="Nets" color="2" fill="1" visible="yes" active="yes"/>
 <layer number="92" name="Busses" color="1" fill="1" visible="yes" active="yes"/>
@@
 <layer number="97" name="Info" color="7" fill="1" visible="yes" active="yes"/>
 <layer number="98" name="Guide" color="6" fill="1" visible="yes" active="yes"/>
+<layer number="99" name="SpiceOrder" color="7" fill="1" visible="yes" active="yes"/>
 <layer number="100" name="Muster" color="7" fill="1" visible="no" active="no"/>
 <layer number="101" name="Patch_Top" color="12" fill="4" visible="no" active="yes"/>
@@
 <layer number="111" name="MPL" color="7" fill="1" visible="yes" active="yes"/>
 <layer number="112" name="tSilk" color="7" fill="1" visible="yes" active="yes"/>
+<layer number="113" name="IDFDebug" color="7" fill="1" visible="no" active="no"/>
+<layer number="114" name="FRNTMAAT1" color="7" fill="1" visible="yes" active="yes"/>
+<layer number="115" name="FRNTMAAT2" color="7" fill="1" visible="yes" active="yes"/>
 <layer number="116" name="Patch_BOT" color="9" fill="4" visible="no" active="yes"/>
+<layer number="117" name="BACKMAAT1" color="7" fill="1" visible="yes" active="yes"/>
+<layer number="118" name="Rect_Pads" color="7" fill="1" visible="no" active="no"/>
+<layer number="119" name="KAP_TEKEN" color="7" fill="1" visible="yes" active="yes"/>
+<layer number="120" name="KAP_MAAT1" color="7" fill="1" visible="yes" active="yes"/>
 <layer number="121" name="_tsilk" color="7" fill="1" visible="no" active="yes"/>
 <layer number="122" name="_bsilk" color="7" fill="1" visible="no" active="yes"/>
@@
 <layer number="127" name="_tValues" color="7" fill="1" visible="yes" active="yes"/>
 <layer number="128" name="_bValues" color="7" fill="1" visible="yes" active="yes"/>
+<layer number="130" name="SMDSTROOK" color="7" fill="1" visible="yes" active="yes"/>
 <layer number="131" name="tAdjust" color="7" fill="1" visible="no" active="yes"/>
 <layer number="132" name="bAdjust" color="7" fill="1" visible="no" active="yes"/>
@@
 <layer number="223" name="223bmp" color="24" fill="1" visible="no" active="no"/>
 <layer number="224" name="224bmp" color="25" fill="1" visible="no" active="no"/>
+<layer number="225" name="225bmp" color="7" fill="1" visible="no" active="no"/>
+<layer number="226" name="226bmp" color="7" fill="1" visible="no" active="no"/>
+<layer number="227" name="227bmp" color="7" fill="1" visible="no" active="no"/>
+<layer number="228" name="228bmp" color="7" fill="1" visible="no" active="no"/>
+<layer number="229" name="229bmp" color="7" fill="1" visible="yes" active="yes"/>
+<layer number="230" name="230bmp" color="7" fill="1" visible="no" active="no"/>
+<layer number="231" name="Eagle3D_PG1" color="7" fill="1" visible="yes" active="yes"/>
+<layer number="232" name="Eagle3D_PG2" color="7" fill="1" visible="yes" active="yes"/>
+<layer number="233" name="Eagle3D_PG3" color="7" fill="1" visible="yes" active="yes"/>
 <layer number="248" name="Housing" color="7" fill="1" visible="yes" active="yes"/>
 <layer number="249" name="Edge" color="7" fill="1" visible="yes" active="yes"/>
@@
 <layer number="251" name="SMDround" color="12" fill="11" visible="no" active="no"/>
 <layer number="254" name="cooling" color="7" fill="1" visible="no" active="yes"/>
+<layer number="255" name="Accent" color="7" fill="1" visible="yes" active="yes"/>
 </layers>
 <schematic xreflabel="%F%N/%S.%C%R" xrefpart="/%S.%C%R">
@@
 <part name="U$20" library="SKAARHOJ" deviceset="GNDPAD" device="6MM" value="GNDPAD6MM"/>
 <part name="U$21" library="SKAARHOJ" deviceset="GNDPAD" device="6MM" value="GNDPAD6MM"/>
-<part name="SERIAL" library="SparkFun" deviceset="M04X2" device=""/>
+<part name="SERIAL" library="SKAARHOJ" deviceset="M04X2" device="M2X4SMALLER"/>
 <part name="GND7" library="SparkFun" deviceset="GND" device=""/>
 <part name="U$17" library="SparkFun" deviceset="5V" device=""/>
@@
 <part name="C14" library="SparkFun" deviceset="CAP" device="0603-CAP" value="100nF"/>
 <part name="GND6" library="SparkFun" deviceset="GND" device=""/>
-<part name="U$19" library="SKAARHOJ" deviceset="3BITADDR" device=""/>
+<part name="U$19" library="SKAARHOJ" deviceset="3BITADDR" device="SMALL" value="3BITADDRSMALL"/>
 <part name="GND8" library="SparkFun" deviceset="GND" device=""/>
 <part name="U$1" library="SKAARHOJ" deviceset="M02X2" device=""/>
@@
 </sheet>
 </sheets>
+<errors>
+</errors>
 </schematic>
 </drawing>
