File: PCBs/PCB-BI8-1x6SC3/PCB-BI8-1x6SC3.sch (EAGLE design)
At the start: 37 parts, among them IC1 MCP23017SS, IC2 PCA9685

Commit message: Updates
Parts:
- SERIAL: value M04X2 -> M04X2M2X4SMALLER; device SparkFun:M04X2 -> SKAARHOJ:M04X2M2X4SMALLER
- U$19: value 3BITADDR -> 3BITADDRSMALL; device SKAARHOJ:3BITADDR -> SKAARHOJ:3BITADDRSMALL
