File: PCBs/PCB-BI8-2x4/PCB-BI8-2x4.brd (EAGLE design)
At the start: 83.8 x 35.6 mm, 37 parts, among them IC1 MCP23017SS, IC2 PCA9685

Commit message: asdf
Parts:
- removed SJ1, SJ2: SOLDERJUMPERNC, SparkFun:SJ_2S
- added U$15, U$18, U$20, U$21: GNDPAD, SKAARHOJ:3.2MMPAD
Connections:
- removed net 5VL: IC1.18, IC2.24, IC2.4, IC2.5, SJ1.2
- removed net GNDL: B1.P$4, B1ALT.P$4, B2.P$4, B2ALT.P$4, B3.P$4, B4.P$4, B4ALT.P$4, B5.P$4, B6.P$4, B7.P$4, B8.P$4, B8ALT.P$4, IC1.1, IC2.23, IC2.25, SJ2.2
- net 5V: now also IC1.18, IC2.24, IC2.4, IC2.5; no longer SJ1.1
- net GND: now also B1.P$4, B1ALT.P$4, B2.P$4, B2ALT.P$4, B3.P$4, B4.P$4, B4ALT.P$4, B5.P$4, B6.P$4, B7.P$4, B8.P$4, B8ALT.P$4, IC1.1, IC2.23, IC2.25, U$15.P$1, U$18.P$1, U$20.P$1, U$21.P$1; no longer SJ2.1
Routing:
- net GND: track 0.00 -> 237.9 mm
- net 5V: track 0.00 -> 229.9 mm, vias 0 -> 3
- net A2: track 0.00 -> 123.0 mm, vias 0 -> 4
- net I2C_SDA: track 0.00 -> 115.1 mm, vias 0 -> 7
- net N$12: track 0.00 -> 114.5 mm, vias 0 -> 2
- net GPA7: track 0.00 -> 108.8 mm, vias 0 -> 2
- net A1: track 0.00 -> 106.3 mm, vias 0 -> 4
- net A0: track 0.00 -> 105.9 mm, vias 0 -> 3
- net I2C_SCL: track 0.00 -> 102.0 mm, vias 0 -> 4
- net GPA0: track 0.00 -> 76.5 mm, vias 0 -> 3
- net GPA6: track 0.00 -> 71.7 mm, vias 0 -> 4
- net N$21: track 0.00 -> 70.0 mm, vias 0 -> 4
- net GPA1: track 0.00 -> 69.1 mm, vias 0 -> 2
- net N$11: track 0.00 -> 65.7 mm, vias 0 -> 2
- net N$10: track 0.00 -> 64.5 mm, vias 0 -> 2
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Other:
- board text added: "PCB-BI8-2x4"
- board text added: "v22-04-13"
- board text removed: "5V"
- board text removed: "BI8-2x4"
- board text removed: "GND"
- board text removed: "v??-??-??"

Commit message: asdf
Routing:
- net N$12: track 114.5 -> 86.0 mm
- net A2: track 123.0 -> 115.3 mm, vias 4 -> 3
- net A1: track 106.3 -> 110.1 mm, vias 4 -> 1
- net GPA7: track 108.8 -> 110.6 mm, vias 2 -> 0
- net A0: track 105.9 -> 104.4 mm, vias 3 -> 5
Other:
- board text added: "v13-05-13"
- board text removed: "v22-04-13"

Commit message: Some work!
Parts:
- U$15, U$18, U$20, U$21: value GNDPAD -> GNDPAD6MM; device SKAARHOJ:3.2MMPAD -> SKAARHOJ:3.2MMPAD6MM
- moved C1 7.65 mm to (11.9, 21.6), turned to 90 degrees
- moved SERIAL 3.67 mm to (76.5, 13.1)
- moved C2 2.54 mm to (74.6, 29.5)
- moved IC2 1.65 mm to (76.8, 23.4)
- moved U$21 1.36 mm to (80.3, 32.1)
- moved U$18 1.36 mm to (80.3, 3.50)
- moved U$20 1.36 mm to (3.50, 32.1)
- moved U$15 1.36 mm to (3.50, 3.50)
- moved IC1 1.30 mm to (5.97, 22.2)
- moved C3 0.18 mm to (76.1, 6.45), turned to 0 degrees
Routing:
- net 5V: track 230.4 -> 200.2 mm
- net GND: track 238.4 -> 217.1 mm
- net GPA7: track 110.6 -> 92.3 mm
- net N$20: track 63.4 -> 81.2 mm
- net N$19: track 64.0 -> 80.9 mm, vias 4 -> 2
- net GPA5: track 62.4 -> 50.9 mm, vias 2 -> 1
- net N$10: track 64.5 -> 53.6 mm, vias 2 -> 4
- net A0: track 104.4 -> 114.7 mm, vias 5 -> 1
- net GPA1: track 69.1 -> 78.9 mm
- net A1: track 110.1 -> 100.5 mm, vias 1 -> 2
- net N$12: track 86.0 -> 78.2 mm, vias 2 -> 4
- net GPA2: track 43.2 -> 50.9 mm
- net I2C_SDA: track 115.1 -> 107.5 mm, vias 7 -> 5
- net N$11: track 65.7 -> 59.2 mm
- net A2: track 115.3 -> 109.9 mm
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- removed copper zone on layer 1, net GND
- removed copper zone on layer 16, net GND

Commit message: Large revisions of boards, change of forms, in particular all mounting holes now has a 7mm diameter and fully inside the board.
Other:
- board text added: "v??-??-??"
- board text removed: "v13-05-13"
Changed lines of the file:
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@@
 <text x="47.244" y="33.4772" size="1.016" layer="122" rot="MR0">PCB-BI8-2x4</text>
 <text x="75.4888" y="33.4772" size="1.524" layer="122" rot="MR0">SKAARHOJ 2013</text>
-<text x="28.702" y="34.29" size="0.8128" layer="122" rot="MR180">v13-05-13</text>
+<text x="28.702" y="34.29" size="0.8128" layer="122" rot="MR180">v??-??-??</text>
 <text x="40.3225" y="1.651" size="0.8128" layer="122" font="vector" rot="MR0">GITHUB: SKAARHOJ-Open-Engineering</text>
 <wire x1="76.454" y1="8.001" x2="73.279" y2="8.001" width="0.4064" layer="122"/>

Commit message: Boards
Routing:
- added copper zone on layer 1, net GND
- added copper zone on layer 16, net GND
Other:
- board text added: "v07-13"
- board text removed: "v??-??-??"
Changed lines of the file:
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@@
 <text x="47.244" y="33.4772" size="1.016" layer="122" rot="MR0">PCB-BI8-2x4</text>
 <text x="75.4888" y="33.4772" size="1.524" layer="122" rot="MR0">SKAARHOJ 2013</text>
-<text x="28.702" y="34.29" size="0.8128" layer="122" rot="MR180">v??-??-??</text>
+<text x="28.702" y="34.29" size="0.8128" layer="122" rot="MR180">v07-13</text>
 <text x="40.3225" y="1.651" size="0.8128" layer="122" font="vector" rot="MR0">GITHUB: SKAARHOJ-Open-Engineering</text>
 <wire x1="76.454" y1="8.001" x2="73.279" y2="8.001" width="0.4064" layer="122"/>
@@
 <wire x1="77.3176" y1="20.9296" x2="70.4088" y2="14.0208" width="0.4064" layer="16"/>
 <wire x1="69.2912" y1="14.0208" x2="69.27" y2="13.97" width="0.4064" layer="16"/>
+<polygon width="0.4064" layer="1">
+<vertex x="0" y="0"/>
+<vertex x="83.82" y="0"/>
+<vertex x="83.82" y="35.56"/>
+<vertex x="0" y="35.56"/>
+</polygon>
+<polygon width="0.4064" layer="16">
+<vertex x="0" y="0"/>
+<vertex x="83.82" y="0"/>
+<vertex x="83.82" y="35.56"/>
+<vertex x="0" y="35.56"/>
+</polygon>
 </signal>
 <signal name="GPA0">

Commit message: PCBS updated
Parts:
- removed C3: 10uF, SparkFun:0805
- added C4: 22uF, SparkFun:0805
- added C5, C6, C7, C8: 100nF, SparkFun:0603-CAP
- added L4: ILHB0805ER121V, SparkFun:0805
Connections:
- new net N$1: C6.1, L4.1, SERIAL.2
- net 5V: now also C4.1, C5.1, C7.1, C8.1, L4.2; no longer C3.1, SERIAL.2
- net GND: now also C4.2, C5.2, C6.2, C7.2, C8.2; no longer C3.2
Routing:
- net GND: track 217.1 -> 291.3 mm, vias 0 -> 10
- net GPA1: track 78.9 -> 58.5 mm, vias 2 -> 1
- net I2C_SCL: track 101.5 -> 119.9 mm, vias 5 -> 6
- net A0: track 114.7 -> 96.5 mm, vias 1 -> 2
- net N$21: track 73.2 -> 56.5 mm
- net 5V: track 200.2 -> 214.8 mm, vias 3 -> 7
- net N$20: track 81.2 -> 66.9 mm
- net GPA5: track 50.9 -> 62.4 mm, vias 1 -> 3
- net GPA4: track 35.3 -> 46.7 mm, vias 1 -> 2
- net N$11: track 59.2 -> 48.8 mm, vias 2 -> 4
- net N$9: track 37.5 -> 46.6 mm, vias 2 -> 4
- net GPA7: track 92.3 -> 84.8 mm, vias 0 -> 1
- net GPA2: track 50.9 -> 43.7 mm, vias 2 -> 0
- net A1: track 100.5 -> 106.9 mm, vias 2 -> 3
- net A2: track 109.9 -> 103.6 mm, vias 3 -> 2
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Other:
- board text added: "SKAARHOJ 2014"
- board text added: "v10-14"
- board text removed: "SKAARHOJ 2013"
- board text removed: "v07-13"

Commit message: PCB updates
Connections:
- net SDI_MOSI renamed SPI_MOSI
- net SDI_SCLK renamed SPI_SCLK
- net SLIDER_IN renamed ANALOG0
- removed net DISP_DATA_OUT: SERIAL.6
Changed lines of the file:
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@@
 <?xml version="1.0" encoding="utf-8"?>
 <!DOCTYPE eagle SYSTEM "eagle.dtd">
-<eagle version="7.1.0">
+<eagle version="7.5.0">
 <drawing>
 <settings>
@@
 <via x="1.7272" y="17.1704" extent="1-16" drill="0.4064"/>
 </signal>
-<signal name="SDI_SCLK">
+<signal name="SPI_SCLK">
 <contactref element="SERIAL" pad="7"/>
 </signal>
-<signal name="SDI_MOSI">
+<signal name="SPI_MOSI">
 <contactref element="SERIAL" pad="8"/>
-</signal>
-<signal name="DISP_DATA_OUT">
-<contactref element="SERIAL" pad="6"/>
-</signal>
-<signal name="SLIDER_IN">
-<contactref element="SERIAL" pad="5"/>
 </signal>
 <signal name="I2C_SDA">
@@
 <wire x1="77.8256" y1="9.2456" x2="77.724" y2="9.271" width="0.4064" layer="16"/>
 </signal>
+<signal name="ANALOG0">
+<contactref element="SERIAL" pad="5"/>
+</signal>
 </signals>

Commit message: Updates
Parts:
- SERIAL: value M04X2 -> M04X2M2X4SMALLER; device SparkFun:2X4 -> SKAARHOJ:M2X4SMALLER
- U$19: value 3BITADDR -> 3BITADDRSMALL; device SKAARHOJ:3BITADDR -> SKAARHOJ:3BITADDR_SMALL
- turned SERIAL to 180 degrees
Connections:
- net 5V: now also U$19.H0; no longer U$19.H3
- net A0: now also U$19.AS0
- net A1: now also U$19.AS1
- net A2: now also U$19.AS2
- net GND: now also U$19.L0; no longer U$19.L3
Routing:
- net GND: track 291.3 -> 329.8 mm
- net A1: track 106.9 -> 108.5 mm, vias 3 -> 4
- net 5V: track 214.8 -> 216.1 mm
- net A2: track 103.6 -> 104.9 mm
Other:
- board text added: "PCB-BI8-2x4, v03-16 SKAARHOJ 2016"
- board text removed: "GITHUB: SKAARHOJ-Open-Engineering"
- board text removed: "PCB-BI8-2x4"
- board text removed: "SKAARHOJ 2014"
- board text removed: "v10-14"
