File: PCBs/PCB-BI8-2x4C3/PCB-BI8-2x4C3.sch (EAGLE design)
At the start: 52 parts, among them IC1 MCP23017SS, IC2 PCA9685

Commit message: ag
Parts:
- removed B10, B10ALT, B11, B11ALT, B12, B12ALT, B13, B14, B15, B16, B5ALT, B6ALT, B7ALT, B9, B9ALT: NKK-NP01-SINGLECOLOR, SKAARHOJ:NKK-NP01-SINGLECOLOR
- added B1ALT, B2ALT: LP11-B", SKAARHOJ:LP11-B"
- B1, B2, B3, B4, B4ALT, B5, B6, B7, B8, B8ALT: value NKK-NP01-SINGLECOLOR -> LP11-B"; device SKAARHOJ:NKK-NP01-SINGLECOLOR -> SKAARHOJ:LP11-B"
- R10, R11, R12, R13, R14, R15, R16, R17, R18, R19, R20, R5, R6, R7, R8, R9: value 100R -> 270
Connections:
- removed net GPB0: B9.SW2, B9ALT.SW2, IC1.GPB0
- removed net GPB1: B10.SW2, B10ALT.SW2, IC1.GPB1
- removed net GPB2: B11.SW2, B11ALT.SW2, IC1.GPB2
- removed net GPB3: B12.SW2, B12ALT.SW2, IC1.GPB3
- removed net GPB4: B13.SW2, IC1.GPB4
- removed net GPB5: B14.SW2, IC1.GPB5
- removed net GPB6: B15.SW2, IC1.GPB6
- removed net GPB7: B16.SW2, IC1.GPB7
- net 5V: now also B1.A, B1ALT.A, B2.A, B2ALT.A, B3.A, B4.A, B4ALT.A, B5.A, B6.A, B7.A, B8.A, B8ALT.A; no longer B1.LC1, B10.LC1, B10ALT.LC1, B11.LC1, B11ALT.LC1, B12.LC1, B12ALT.LC1, B13.LC1, B14.LC1, B15.LC1, B16.LC1, B2.LC1, B3.LC1, B4.LC1, B4ALT.LC1, B5.LC1, B5ALT.LC1, B6.LC1, B6ALT.LC1, B7.LC1, B7ALT.LC1, B8.LC1, B8ALT.LC1, B9.LC1, B9ALT.LC1
- net GND: now also B1ALT.SW1, B2ALT.SW1, IC1.GPB0; no longer B10.SW1, B10ALT.SW1, B11.SW1, B11ALT.SW1, B12.SW1, B12ALT.SW1, B13.SW1, B14.SW1, B15.SW1, B16.SW1, B5ALT.SW1, B6ALT.SW1, B7ALT.SW1, B9.SW1, B9ALT.SW1
- net GPA0: now also B8.SW2, B8ALT.SW2; no longer B1.SW2
- net GPA1: now also B7.SW2; no longer B2.SW2
- net GPA2: now also B6.SW2; no longer B3.SW2
- net GPA3: now also B5.SW2; no longer B4.SW2, B4ALT.SW2
- net GPA4: now also B1.SW2, B1ALT.SW2; no longer B5.SW2, B5ALT.SW2
- net GPA5: now also B2.SW2, B2ALT.SW2; no longer B6.SW2, B6ALT.SW2
- net GPA6: now also B3.SW2; no longer B7.SW2, B7ALT.SW2
- net GPA7: now also B4.SW2, B4ALT.SW2; no longer B8.SW2, B8ALT.SW2
- net L0: now also B1.K1, B1ALT.K1; no longer B1.L1, B1.L2
- net L1: now also B1.K2, B1ALT.K2; no longer B2.L1, B2.L2
- net L10: now also B6.K1; no longer B11.L1, B11.L2, B11ALT.L1, B11ALT.L2
- net L11: now also B6.K2; no longer B12.L1, B12.L2, B12ALT.L1, B12ALT.L2
- net L12: now also B7.K1; no longer B13.L1, B13.L2
- net L13: now also B7.K2; no longer B14.L1, B14.L2
- net L14: now also B8.K1, B8ALT.K1; no longer B15.L1, B15.L2
- net L15: now also B8.K2, B8ALT.K2; no longer B16.L1, B16.L2
- net L2: now also B2.K1, B2ALT.K1; no longer B3.L1, B3.L2
- net L3: now also B2.K2, B2ALT.K2; no longer B4.L1, B4.L2, B4ALT.L1, B4ALT.L2
- net L4: now also B3.K1; no longer B5.L1, B5.L2, B5ALT.L1, B5ALT.L2
- net L5: now also B3.K2; no longer B6.L1, B6.L2, B6ALT.L1, B6ALT.L2
- net L6: now also B4.K1, B4ALT.K1; no longer B7.L1, B7.L2, B7ALT.L1, B7ALT.L2
- net L7: now also B4.K2, B4ALT.K2; no longer B8.L1, B8.L2, B8ALT.L1, B8ALT.L2
- net L8: now also B5.K1; no longer B9.L1, B9.L2, B9ALT.L1, B9ALT.L2
- net L9: now also B5.K2; no longer B10.L1, B10.L2, B10ALT.L1, B10ALT.L2

Commit message: PCBS updated
Parts:
- removed C3: 10uF, SparkFun:CAP0805
- added C4: 22uF, SparkFun:CAP0805
- added C5, C6, C7, C8: 100nF, SparkFun:CAP0603-CAP
- added L4: ILHB0805ER121V, SparkFun:INDUCTOR0805
Connections:
- new net N$1: C6.1, L4.1, SERIAL.2
- net 5V: now also C4.1, C5.1, C7.1, C8.1, L4.2; no longer C3.1, SERIAL.2
- net GND: now also C4.2, C5.2, C6.2, C7.2, C8.2; no longer C3.2
Other:
- note removed: "POWER"

Commit message: PCB updates
Parts:
- U$19: value 3BITADDR -> 3BITADDRSMALL; device SKAARHOJ:3BITADDR -> SKAARHOJ:3BITADDRSMALL

Commit message: Updates
Parts:
- SERIAL: value M04X2 -> M04X2M2X4SMALLER; device SparkFun:M04X2 -> SKAARHOJ:M04X2M2X4SMALLER
Changed lines of the file:
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@@
 <grid distance="0.1" unitdist="inch" unit="inch" style="lines" multiple="1" display="no" altdistance="0.01" altunitdist="inch" altunit="inch"/>
 <layers>
-<layer number="1" name="Top" color="4" fill="1" visible="yes" active="no"/>
-<layer number="2" name="Route2" color="1" fill="3" visible="yes" active="no"/>
-<layer number="3" name="Route3" color="4" fill="3" visible="yes" active="no"/>
-<layer number="4" name="Route4" color="1" fill="4" visible="yes" active="no"/>
-<layer number="5" name="Route5" color="4" fill="4" visible="yes" active="no"/>
-<layer number="6" name="Route6" color="1" fill="8" visible="yes" active="no"/>
-<layer number="7" name="Route7" color="4" fill="8" visible="yes" active="no"/>
-<layer number="8" name="Route8" color="1" fill="2" visible="yes" active="no"/>
-<layer number="9" name="Route9" color="4" fill="2" visible="yes" active="no"/>
-<layer number="10" name="Route10" color="1" fill="7" visible="yes" active="no"/>
-<layer number="11" name="Route11" color="4" fill="7" visible="yes" active="no"/>
-<layer number="12" name="Route12" color="1" fill="5" visible="yes" active="no"/>
-<layer number="13" name="Route13" color="4" fill="5" visible="yes" active="no"/>
-<layer number="14" name="Route14" color="1" fill="6" visible="yes" active="no"/>
-<layer number="15" name="Route15" color="4" fill="6" visible="yes" active="no"/>
-<layer number="16" name="Bottom" color="1" fill="1" visible="yes" active="no"/>
-<layer number="17" name="Pads" color="2" fill="1" visible="yes" active="no"/>
-<layer number="18" name="Vias" color="2" fill="1" visible="yes" active="no"/>
-<layer number="19" name="Unrouted" color="13" fill="1" visible="yes" active="no"/>
-<layer number="20" name="Dimension" color="15" fill="1" visible="yes" active="no"/>
-<layer number="21" name="tPlace" color="7" fill="1" visible="yes" active="no"/>
-<layer number="22" name="bPlace" color="7" fill="1" visible="yes" active="no"/>
-<layer number="23" name="tOrigins" color="15" fill="1" visible="yes" active="no"/>
-<layer number="24" name="bOrigins" color="15" fill="1" visible="yes" active="no"/>
-<layer number="25" name="tNames" color="7" fill="1" visible="yes" active="no"/>
-<layer number="26" name="bNames" color="7" fill="1" visible="yes" active="no"/>
-<layer number="27" name="tValues" color="7" fill="1" visible="yes" active="no"/>
-<layer number="28" name="bValues" color="7" fill="1" visible="yes" active="no"/>
+<layer number="1" name="Top" color="4" fill="1" visible="no" active="no"/>
+<layer number="2" name="Route2" color="1" fill="3" visible="no" active="no"/>
+<layer number="3" name="Route3" color="4" fill="3" visible="no" active="no"/>
+<layer number="4" name="Route4" color="1" fill="4" visible="no" active="no"/>
+<layer number="5" name="Route5" color="4" fill="4" visible="no" active="no"/>
+<layer number="6" name="Route6" color="1" fill="8" visible="no" active="no"/>
+<layer number="7" name="Route7" color="4" fill="8" visible="no" active="no"/>
+<layer number="8" name="Route8" color="1" fill="2" visible="no" active="no"/>
+<layer number="9" name="Route9" color="4" fill="2" visible="no" active="no"/>
+<layer number="10" name="Route10" color="1" fill="7" visible="no" active="no"/>
+<layer number="11" name="Route11" color="4" fill="7" visible="no" active="no"/>
+<layer number="12" name="Route12" color="1" fill="5" visible="no" active="no"/>
+<layer number="13" name="Route13" color="4" fill="5" visible="no" active="no"/>
+<layer number="14" name="Route14" color="1" fill="6" visible="no" active="no"/>
+<layer number="15" name="Route15" color="4" fill="6" visible="no" active="no"/>
+<layer number="16" name="Bottom" color="1" fill="1" visible="no" active="no"/>
+<layer number="17" name="Pads" color="2" fill="1" visible="no" active="no"/>
+<layer number="18" name="Vias" color="2" fill="1" visible="no" active="no"/>
+<layer number="19" name="Unrouted" color="13" fill="1" visible="no" active="no"/>
+<layer number="20" name="Dimension" color="15" fill="1" visible="no" active="no"/>
+<layer number="21" name="tPlace" color="7" fill="1" visible="no" active="no"/>
+<layer number="22" name="bPlace" color="7" fill="1" visible="no" active="no"/>
+<layer number="23" name="tOrigins" color="15" fill="1" visible="no" active="no"/>
+<layer number="24" name="bOrigins" color="15" fill="1" visible="no" active="no"/>
+<layer number="25" name="tNames" color="7" fill="1" visible="no" active="no"/>
+<layer number="26" name="bNames" color="7" fill="1" visible="no" active="no"/>
+<layer number="27" name="tValues" color="7" fill="1" visible="no" active="no"/>
+<layer number="28" name="bValues" color="7" fill="1" visible="no" active="no"/>
 <layer number="29" name="tStop" color="7" fill="3" visible="no" active="no"/>
 <layer number="30" name="bStop" color="7" fill="6" visible="no" active="no"/>
@@
 <layer number="35" name="tGlue" color="7" fill="4" visible="no" active="no"/>
 <layer number="36" name="bGlue" color="7" fill="5" visible="no" active="no"/>
-<layer number="37" name="tTest" color="7" fill="1" visible="yes" active="no"/>
-<layer number="38" name="bTest" color="7" fill="1" visible="yes" active="no"/>
+<layer number="37" name="tTest" color="7" fill="1" visible="no" active="no"/>
+<layer number="38" name="bTest" color="7" fill="1" visible="no" active="no"/>
 <layer number="39" name="tKeepout" color="4" fill="11" visible="no" active="no"/>
 <layer number="40" name="bKeepout" color="1" fill="11" visible="no" active="no"/>
@@
 <layer number="44" name="Drills" color="7" fill="1" visible="no" active="no"/>
 <layer number="45" name="Holes" color="7" fill="1" visible="no" active="no"/>
-<layer number="46" name="Milling" color="3" fill="1" visible="yes" active="no"/>
-<layer number="47" name="Measures" color="7" fill="1" visible="yes" active="no"/>
-<layer number="48" name="Document" color="7" fill="1" visible="yes" active="no"/>
-<layer number="49" name="Reference" color="7" fill="1" visible="yes" active="no"/>
-<layer number="50" name="dxf" color="7" fill="1" visible="yes" active="no"/>
-<layer number="51" name="tDocu" color="7" fill="1" visible="yes" active="no"/>
-<layer number="52" name="bDocu" color="7" fill="1" visible="yes" active="no"/>
-<layer number="53" name="tGND_GNDA" color="7" fill="9" visible="yes" active="no"/>
-<layer number="54" name="bGND_GNDA" color="1" fill="9" visible="yes" active="no"/>
-<layer number="56" name="wert" color="7" fill="1" visible="yes" active="no"/>
-<layer number="57" name="tCAD" color="7" fill="1" visible="yes" active="no"/>
+<layer number="46" name="Milling" color="3" fill="1" visible="no" active="no"/>
+<layer number="47" name="Measures" color="7" fill="1" visible="no" active="no"/>
+<layer number="48" name="Document" color="7" fill="1" visible="no" active="no"/>
+<layer number="49" name="Reference" color="7" fill="1" visible="no" active="no"/>
+<layer number="50" name="dxf" color="7" fill="1" visible="no" active="no"/>
+<layer number="51" name="tDocu" color="7" fill="1" visible="no" active="no"/>
+<layer number="52" name="bDocu" color="7" fill="1" visible="no" active="no"/>
+<layer number="53" name="tGND_GNDA" color="7" fill="9" visible="no" active="no"/>
+<layer number="54" name="bGND_GNDA" color="1" fill="9" visible="no" active="no"/>
+<layer number="56" name="wert" color="7" fill="1" visible="no" active="no"/>
+<layer number="57" name="tCAD" color="7" fill="1" visible="no" active="no"/>
 <layer number="90" name="Modules" color="5" fill="1" visible="yes" active="yes"/>
 <layer number="91" name="Nets" color="2" fill="1" visible="yes" active="yes"/>
@@
 <part name="B8ALT" library="SKAARHOJ" deviceset="LP11-B" device="&quot;"/>
 <part name="U$16" library="SparkFun" deviceset="5V" device=""/>
-<part name="SERIAL" library="SparkFun" deviceset="M04X2" device=""/>
+<part name="SERIAL" library="SKAARHOJ" deviceset="M04X2" device="M2X4SMALLER"/>
 <part name="GND5" library="SparkFun" deviceset="GND" device=""/>
 <part name="B2ALT" library="SKAARHOJ" deviceset="LP11-B" device="&quot;"/>
