File: PCBs/PCB-SSB-2x1/PCB-SSB-2x1.sch (EAGLE design)
At the start: 12 parts, among them IC1 MCP23017SS

Commit message: asdf
Parts:
- removed R1, R2: 10K, SparkFun:RESISTOR0603-RES
- removed RN1: 10K, SKAARHOJ:4R-NCAY16
- removed S2: SWS003, smd-special:SWS003
- removed SJ1, SJ2: SOLDERJUMPERNC, SparkFun:SOLDERJUMPERNC
- added U$15, U$18, U$20, U$21: GNDPAD, SKAARHOJ:GNDPAD
- added U$19: 3BITADDR, SKAARHOJ:3BITADDR
Connections:
- removed net 5VL: IC1.!RESET, R1.1, R2.1, S2.1, S2.2, S2.3, SJ1.2
- removed net GNDL: RN1A.1, RN1B.1, RN1C.1, RN1D.1, SJ2.2
- net 5V: now also IC1.!RESET, U$19.VCC; no longer SJ1.1
- net A0: now also U$19.A0; no longer RN1D.2, S2.6
- net A1: now also U$19.A1; no longer RN1C.2, S2.5
- net A2: now also U$19.A2; no longer RN1B.2, S2.4
- net GND: now also U$15.1, U$18.1, U$19.GND, U$20.1, U$21.1; no longer SJ2.1
- net I2C_SCL: no longer R2.2
- net I2C_SDA: no longer R1.2

Commit message: Large revisions of boards, change of forms, in particular all mounting holes now has a 7mm diameter and fully inside the board.
Parts:
- removed U$20, U$21: GNDPAD, SKAARHOJ:GNDPAD
- U$15, U$18: value GNDPAD -> GNDPAD6MM; device SKAARHOJ:GNDPAD -> SKAARHOJ:GNDPAD6MM
- renumbered U$2 to SSW1, U$3 to SSW2
Connections:
- net GND: no longer U$20.1, U$21.1
Changed lines of the file:
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@@
 <part name="GND5" library="SparkFun" deviceset="GND" device=""/>
 <part name="U$17" library="SparkFun" deviceset="5V" device=""/>
-<part name="U$2" library="SKAARHOJ" deviceset="SMART_SWITCH" device="SMART_SWITCH_8PIN"/>
-<part name="U$3" library="SKAARHOJ" deviceset="SMART_SWITCH" device="SMART_SWITCH_8PIN"/>
+<part name="SSW1" library="SKAARHOJ" deviceset="SMART_SWITCH" device="SMART_SWITCH_8PIN"/>
+<part name="SSW2" library="SKAARHOJ" deviceset="SMART_SWITCH" device="SMART_SWITCH_8PIN"/>
 <part name="U$19" library="SKAARHOJ" deviceset="3BITADDR" device=""/>
-<part name="U$15" library="SKAARHOJ" deviceset="GNDPAD" device=""/>
-<part name="U$18" library="SKAARHOJ" deviceset="GNDPAD" device=""/>
-<part name="U$20" library="SKAARHOJ" deviceset="GNDPAD" device=""/>
-<part name="U$21" library="SKAARHOJ" deviceset="GNDPAD" device=""/>
+<part name="U$15" library="SKAARHOJ" deviceset="GNDPAD" device="6MM" value="GNDPAD6MM"/>
+<part name="U$18" library="SKAARHOJ" deviceset="GNDPAD" device="6MM" value="GNDPAD6MM"/>
 </parts>
 <sheets>
@@
 <instance part="GND5" gate="1" x="48.26" y="-2.54"/>
 <instance part="U$17" gate="G$1" x="71.12" y="15.24"/>
-<instance part="U$2" gate="G$1" x="-40.64" y="88.9"/>
-<instance part="U$3" gate="G$1" x="7.62" y="88.9"/>
+<instance part="SSW1" gate="G$1" x="-40.64" y="88.9"/>
+<instance part="SSW2" gate="G$1" x="7.62" y="88.9"/>
 <instance part="U$19" gate="G$1" x="-10.16" y="5.08"/>
 <instance part="U$15" gate="G$1" x="50.8" y="-22.86"/>
 <instance part="U$18" gate="G$1" x="78.74" y="-22.86"/>
-<instance part="U$20" gate="G$1" x="50.8" y="-35.56"/>
-<instance part="U$21" gate="G$1" x="78.74" y="-35.56"/>
 </instances>
 <busses>
@@
 </segment>
 <segment>
-<pinref part="U$2" gate="G$1" pin="VDD"/>
+<pinref part="SSW1" gate="G$1" pin="VDD"/>
 <wire x1="-53.34" y1="86.36" x2="-55.88" y2="86.36" width="0.1524" layer="91"/>
 <label x="-55.88" y="86.36" size="1.778" layer="95" rot="R180"/>
 </segment>
 <segment>
-<pinref part="U$3" gate="G$1" pin="VDD"/>
+<pinref part="SSW2" gate="G$1" pin="VDD"/>
 <wire x1="-5.08" y1="86.36" x2="-7.62" y2="86.36" width="0.1524" layer="91"/>
 <label x="-7.62" y="86.36" size="1.778" layer="95" rot="R180"/>
@@
 </segment>
 <segment>
-<pinref part="U$2" gate="G$1" pin="GND"/>
+<pinref part="SSW1" gate="G$1" pin="GND"/>
 <wire x1="-53.34" y1="83.82" x2="-55.88" y2="83.82" width="0.1524" layer="91"/>
-<pinref part="U$2" gate="G$1" pin="SW1"/>
+<pinref part="SSW1" gate="G$1" pin="SW1"/>
 <wire x1="-53.34" y1="78.74" x2="-55.88" y2="78.74" width="0.1524" layer="91"/>
 <wire x1="-55.88" y1="83.82" x2="-55.88" y2="78.74" width="0.1524" layer="91"/>
@@
 </segment>
 <segment>
-<pinref part="U$3" gate="G$1" pin="GND"/>
+<pinref part="SSW2" gate="G$1" pin="GND"/>
 <wire x1="-5.08" y1="83.82" x2="-7.62" y2="83.82" width="0.1524" layer="91"/>
-<pinref part="U$3" gate="G$1" pin="SW1"/>
+<pinref part="SSW2" gate="G$1" pin="SW1"/>
 <wire x1="-5.08" y1="78.74" x2="-7.62" y2="78.74" width="0.1524" layer="91"/>
 <wire x1="-7.62" y1="83.82" x2="-7.62" y2="78.74" width="0.1524" layer="91"/>
@@
 <label x="88.9" y="-22.86" size="1.778" layer="95"/>
 </segment>
-<segment>
-<pinref part="U$20" gate="G$1" pin="1"/>
-<wire x1="55.88" y1="-35.56" x2="60.96" y2="-35.56" width="0.1524" layer="91"/>
-<label x="60.96" y="-35.56" size="1.778" layer="95"/>
-</segment>
-<segment>
-<pinref part="U$21" gate="G$1" pin="1"/>
-<wire x1="83.82" y1="-35.56" x2="88.9" y2="-35.56" width="0.1524" layer="91"/>
-<label x="88.9" y="-35.56" size="1.778" layer="95"/>
-</segment>
 </net>
 <net name="GPA0" class="0">
@@
 </segment>
 <segment>
-<pinref part="U$2" gate="G$1" pin="SW2"/>
+<pinref part="SSW1" gate="G$1" pin="SW2"/>
 <wire x1="-27.94" y1="78.74" x2="-25.4" y2="78.74" width="0.1524" layer="91"/>
 <label x="-25.4" y="78.74" size="1.778" layer="95"/>
@@
 </segment>
 <segment>
-<pinref part="U$3" gate="G$1" pin="SW2"/>
+<pinref part="SSW2" gate="G$1" pin="SW2"/>
 <wire x1="20.32" y1="78.74" x2="22.86" y2="78.74" width="0.1524" layer="91"/>
 <label x="22.86" y="78.74" size="1.778" layer="95"/>
@@
 </segment>
 <segment>
-<pinref part="U$2" gate="G$1" pin="SCK"/>
+<pinref part="SSW1" gate="G$1" pin="SCK"/>
 <wire x1="-53.34" y1="93.98" x2="-55.88" y2="93.98" width="0.1524" layer="91"/>
 <label x="-55.88" y="93.98" size="1.778" layer="95" rot="R180"/>
 </segment>
 <segment>
-<pinref part="U$3" gate="G$1" pin="SCK"/>
+<pinref part="SSW2" gate="G$1" pin="SCK"/>
 <wire x1="-5.08" y1="93.98" x2="-7.62" y2="93.98" width="0.1524" layer="91"/>
 <label x="-7.62" y="93.98" size="1.778" layer="95" rot="R180"/>
@@
 </segment>
 <segment>
-<pinref part="U$2" gate="G$1" pin="SDI"/>
+<pinref part="SSW1" gate="G$1" pin="SDI"/>
 <wire x1="-53.34" y1="91.44" x2="-55.88" y2="91.44" width="0.1524" layer="91"/>
 <label x="-55.88" y="91.44" size="1.778" layer="95" rot="R180"/>
 </segment>
 <segment>
-<pinref part="U$3" gate="G$1" pin="SDI"/>
+<pinref part="SSW2" gate="G$1" pin="SDI"/>
 <wire x1="-5.08" y1="91.44" x2="-7.62" y2="91.44" width="0.1524" layer="91"/>
 <label x="-7.62" y="91.44" size="1.778" layer="95" rot="R180"/>
@@
 </segment>
 <segment>
-<pinref part="U$3" gate="G$1" pin="SS"/>
+<pinref part="SSW2" gate="G$1" pin="SS"/>
 <wire x1="-5.08" y1="96.52" x2="-7.62" y2="96.52" width="0.1524" layer="91"/>
 <label x="-7.62" y="96.52" size="1.778" layer="95" rot="R180"/>
@@
 </segment>
 <segment>
-<pinref part="U$2" gate="G$1" pin="SS"/>
+<pinref part="SSW1" gate="G$1" pin="SS"/>
 <wire x1="-53.34" y1="96.52" x2="-55.88" y2="96.52" width="0.1524" layer="91"/>
 <label x="-55.88" y="96.52" size="1.778" layer="95" rot="R180"/>

Commit message: Updates
Parts:
- SERIAL: value M04X2 -> M04X2M2X4SMALLER; device SparkFun:M04X2 -> SKAARHOJ:M04X2M2X4SMALLER
- U$19: value 3BITADDR -> 3BITADDRSMALL; device SKAARHOJ:3BITADDR -> SKAARHOJ:3BITADDRSMALL
