File: PCBs/PCB-B4LinkMicroS/PCB-B4LinkMicroS.brd (EAGLE design)
At the start: 43.5 x 19.5 mm, 35 parts, among them IC5 LM358D, K1 RELAY5VIM03, Q1 SMD-MOSFET-P-CH-8V-4.1A(SOT-2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, X1 MSTBV33.5MM

Commit message: Updates
Parts:
- R9: value 12K5 -> 22K
Changed lines of the file:
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@@
 <element name="C7" library="SparkFun" package="0603-CAP" value="100nF" x="33.59" y="17.445" rot="MR270"/>
 <element name="C15" library="SparkFun" package="0805" value="10uF/25V" x="31.496" y="17.526" rot="MR270"/>
-<element name="R9" library="SparkFun" package="0603-RES" value="12K5" x="29.083" y="9.271" rot="MR270"/>
+<element name="R9" library="SparkFun" package="0603-RES" value="22K" x="29.083" y="9.271" rot="MR270"/>
 <element name="R10" library="SparkFun" package="0603-RES" value="22K" x="26.924" y="9.271" rot="MR270"/>
 <element name="LED1" library="SKAARHOJ" package="LEDBICOLOR-SMD" value="LEDBICOLOR-SMD" x="4.5" y="15.59" rot="R270"/>
