File: PCBs/PCB-BI8-1x12SC3/PCB-BI8-1x12SC3.brd (EAGLE design)
At the start: 218.4 x 33 mm, 67 parts, among them IC2 PCA9685, IC3 PCA9685, IC4 MCP23017SS

Commit message: asdf
Parts:
- R10, R11, R12, R13, R14, R15, R16, R17, R18, R19, R20, R25, R26, R27, R28, R29, R30, R31, R32, R5, R6, R7, R8, R9: device OPL:R0603 -> SparkFun-Passives:0603-RES
- moved B4ALT 71.1 mm to (149.9, 16.5)
- moved L1 71.1 mm to (181.6, 4.45)
- moved R17 71.1 mm to (195.6, 14.6)
- moved R18 71.1 mm to (195.6, 18.4)
- moved B1 71.1 mm to (210.8, 16.5)
- moved B10 71.1 mm to (50.8, 16.5)
- moved B10ALT 71.1 mm to (43.2, 16.5)
- moved B11 71.1 mm to (33.0, 16.5)
- moved B11ALT 71.1 mm to (25.4, 16.5)
- moved B12 71.1 mm to (15.2, 16.5)
- moved B12ALT 71.1 mm to (7.62, 16.5)
- moved B5ALT 71.1 mm to (132.1, 16.5)
- moved B6 71.1 mm to (121.9, 16.5)
- moved B6ALT 71.1 mm to (114.3, 16.5)
- moved B7 71.1 mm to (104.1, 16.5)
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
Commit message: Fix Encoder bug on EADOGM disp
Changed lines of the file:
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@@
 <?xml version="1.0" encoding="utf-8"?>
 <!DOCTYPE eagle SYSTEM "eagle.dtd">
-<eagle version="7.1.0">
+<eagle version="7.2.0">
 <drawing>
 <settings>

Commit message: asdf
Changed lines of the file:
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@@
 <?xml version="1.0" encoding="utf-8"?>
 <!DOCTYPE eagle SYSTEM "eagle.dtd">
-<eagle version="7.2.0">
+<eagle version="7.1.0">
 <drawing>
 <settings>

Commit message: asdf
Parts:
- removed L2, L3, L4: F.Bead, OPL:L0603
- added C3: 22uF, SparkFun:0805
- added C8, C9: 100nF, SparkFun:0603-CAP
- L1: value F.BEAD -> ILHB0805ER121V; device OPL:L0805 -> SparkFun:0805
- moved L1 1.58 mm to (181.8, 6.02), turned to 180 degrees
- moved PC2 0.63 mm to (186.7, 3.96)
Connections:
- removed net N$17: B5.COM, B5ALT.COM, B6.COM, B6ALT.COM, B7.COM, B7ALT.COM, B8.COM, B8ALT.COM, C1.2, L2.1
- removed net N$18: B1.COM, B1ALT.COM, B2.COM, B3.COM, B4.COM, B4ALT.COM, C6.2, L3.1
- removed net N$29: B10.COM, B10ALT.COM, B11.COM, B11ALT.COM, B12.COM, B12ALT.COM, B9.COM, C7.2, L4.1
- net 5V: now also B1.COM, B10.COM, B10ALT.COM, B11.COM, B11ALT.COM, B12.COM, B12ALT.COM, B1ALT.COM, B2.COM, B3.COM, B4.COM, B4ALT.COM, B5.COM, B5ALT.COM, B6.COM, B6ALT.COM, B7.COM, B7ALT.COM, B8.COM, B8ALT.COM, B9.COM, C1.2, C3.1, C6.2, C7.2, C8.1; no longer L2.2, L3.2, L4.2
- net GND: now also C3.2, C8.2, C9.2
- net N$16: now also C9.1
Routing:
- net 5V: track 221.1 -> 366.0 mm, vias 9 -> 7
- net N$29: track 94.7 -> 0.00 mm
- net N$27: track 108.4 -> 193.9 mm, vias 4 -> 10
- net N$18: track 73.6 -> 0.00 mm, vias 3 -> 0
- net N$17: track 71.1 -> 0.00 mm
- net GPA2: track 131.9 -> 69.9 mm, vias 0 -> 4
- net N$25: track 95.2 -> 123.5 mm, vias 6 -> 4
- net N$21: track 92.4 -> 69.6 mm, vias 2 -> 4
- net N$1: track 68.5 -> 49.3 mm, vias 0 -> 2
- net N$9: track 31.8 -> 14.4 mm, vias 4 -> 2
- net I2C_SCL: track 154.6 -> 171.4 mm
- net GPA15: track 172.6 -> 189.1 mm, vias 4 -> 5
- net A2: track 189.5 -> 176.6 mm, vias 5 -> 11
- net N$11: track 12.1 -> 24.3 mm, vias 0 -> 2
- net N$23: track 89.2 -> 77.2 mm
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Other:
- board text added: "SKAARHOJ 2015"
- board text added: "v04-15"
- board text removed: "SKAARHOJ 2014"
- board text removed: "v10-14"

Commit message: Updates
Parts:
- SERIAL: value M04X2 -> M04X2M2X4SMALLER; device SparkFun:2X4 -> SKAARHOJ:M2X4SMALLER
- U$19: value 3BITADDR -> 3BITADDRSMALL; device SKAARHOJ:3BITADDR -> SKAARHOJ:3BITADDR_SMALL
- turned SERIAL to 90 degrees
Connections:
- net 5V: now also U$19.H0; no longer U$19.H3
- net A0: now also U$19.AS0
- net A1: now also U$19.AS1
- net A2: now also U$19.AS2
- net GND: now also U$19.L0; no longer U$19.L3
Routing:
- net A2: track 176.6 -> 181.6 mm
- net A0: track 148.7 -> 150.2 mm, vias 8 -> 10
- net GND: track 462.9 -> 463.8 mm, vias 7 -> 8
- net A1: track 167.3 -> 168.0 mm, vias 4 -> 6
Other:
- board text added: "PCB-BI8-1x12SC3, v03-16"
- board text removed: "BI8-1x12SC3"
- board text removed: "Github: SKAARHOJ-Open-Engineering"
- board text removed: "SKAARHOJ 2015"
- board text removed: "v04-15"
