File: PCBs/PCB-BI8-2x5RGB/PCB-BI8-2x5RGB.brd (EAGLE design)
At the start: 99.1 x 35.6 mm, 59 parts, among them IC1 MCP23017SS, IC2 PCA9685, IC3 PCA9685

Commit message: Boards
Routing:
- added copper zone on layer 1, net GND
- added copper zone on layer 16, net GND
Other:
- board text added: "v07-13"
- board text removed: "v??-??-??"
