File: PCBs/PCB-E21-CMB6/PCB-E21-CMB6.brd (EAGLE design)
At the start: 200 x 99.5 mm, 172 parts, among them IC1 MCP23017SS, IC2 PCA9685, IC3 PCA9685, IC4 MCP23017SS, IC5 74HCT14D, IC6 PCA9685, IC7 MCP23017SS, IC8 PCA9685, SW1 EC12E_SWCAR1

Commit message: Updates
Parts:
- added U$94: M04X2ZIF-0.5, SKAARHOJ:ZIP-8-0.5
- moved PC1 30.1 mm to (144.8, 54.6), flipped to the bottom
- moved POT1ALT 7.50 mm to (146.0, 63.0)
- flipped PC2 to the bottom
Connections:
- net 5V: now also U$94.P$2
- net GND: now also U$94.P$1
- net I2C_SCL: now also U$94.P$4
- net I2C_SDA: now also U$94.P$3
- net MOSI: now also U$94.P$8
- net SCLK: now also U$94.P$7
Routing:
- net N$53: track 28.2 -> 110.9 mm, vias 0 -> 4
- net SCLK: track 130.8 -> 172.3 mm, vias 5 -> 6
- net 5V: track 967.7 -> 995.2 mm, vias 8 -> 11
- net GND: track 1055.5 -> 1082.5 mm
- net L12: track 162.0 -> 188.5 mm, vias 3 -> 2
- net MOSI: track 150.5 -> 168.1 mm, vias 4 -> 3
- net I2C_SCL: track 390.3 -> 399.8 mm, vias 27 -> 28
- net GPA1: track 272.0 -> 277.4 mm, vias 7 -> 9
- net A0: track 137.5 -> 133.7 mm
- net I2C_SDA: track 331.2 -> 334.0 mm, vias 18 -> 19
- net GPA4: track 70.0 -> 72.7 mm
- net L17: track 136.1 -> 138.0 mm, vias 1 -> 3
- net GPA12: track 208.2 -> 210.0 mm
- net N$52: track 43.3 -> 44.3 mm
- added copper zone on layer 1, net GND
- removed copper zone on layer 1, net N$1
Other:
- outline, holes or cut-outs redrawn
- board text added: "PCB-E21-CMB6, v03-16 SKAARHOJ"
- board text removed: "PCB-E21-CMB6, v02-16 SKAARHOJ"
