File: PCBs/PCB-E21-KP01/PCB-E21-KP01.brd (EAGLE design)
At the start: 99.1 x 74 mm, 69 parts, among them IC1 MCP23017SS, IC2 PCA9685, IC3 PCA9685, IC4 MCP23017SS, IC5 74HCT14D, SW1 EC12E_SWCAR1

Commit message: Updates
Parts:
- added C13: 22uF, SparkFun:0805
- added U$21: M04X2ZIF-0.5, SKAARHOJ:ZIP-8-0.5
- C3, C4: value 10uF -> 22uF
- moved C3 54.3 mm to (64.8, 24.1)
- moved C4 5.08 mm to (33.0, 69.8)
Connections:
- net 5V: now also C13.1, U$21.P$2
- net GND: now also C13.2, U$21.P$1
- net I2C_SCL: now also U$21.P$4
- net I2C_SDA: now also U$21.P$3
- net MOSI: now also U$21.P$8
- net SCLK: now also U$21.P$7
Routing:
- net I2C_SCL: track 147.2 -> 165.6 mm, vias 4 -> 6
- net MOSI: track 35.7 -> 53.6 mm, vias 1 -> 2
- net GND: track 431.7 -> 448.7 mm, vias 21 -> 20
- net SCLK: track 20.7 -> 36.5 mm, vias 1 -> 2
- net I2C_SDA: track 128.0 -> 138.0 mm
- net GPA4S: track 50.1 -> 57.8 mm, vias 1 -> 0
- net 5V: track 426.5 -> 433.2 mm, vias 13 -> 12
- net GPB4: track 60.9 -> 57.5 mm
Other:
- board text added: "PCB-E21-KP01, v03-16 SKAARHOJ"
- board text removed: "PCB-E21-KP01, v02-16 SKAARHOJ"
