File: PCBs/PCB-E21-TVS/PCB-E21-TVS.brd (EAGLE design)
At the start: 120 x 73.7 mm, 48 parts, among them IC3 PCA9685, IC4 MCP23017SS

Commit message: Updates
Parts:
- POT1: device SKAARHOJ:SLIDER20 -> SKAARHOJ:SLIDER20-CAR2
- moved C7 7.85 mm to (68.9, 55.0), turned to 90 degrees
- moved C4 4.34 mm to (91.9, 49.3)
- moved IC4 3.77 mm to (91.0, 43.5)
Routing:
- net GND: track 415.8 -> 436.9 mm, vias 19 -> 20
- net 5V: track 309.2 -> 322.2 mm
- net GPB3: track 21.8 -> 29.2 mm, vias 0 -> 1
- net SLIDER_IN: track 72.3 -> 67.0 mm
- net GPB4: track 41.4 -> 37.4 mm
- net GPB5: track 22.2 -> 18.2 mm
- net GPA0: track 125.1 -> 128.9 mm
- net GPB6: track 55.3 -> 58.9 mm, vias 0 -> 2
- net GPA3: track 57.9 -> 54.4 mm
- net GPA4: track 57.9 -> 54.4 mm
- net GPA5: track 33.2 -> 29.7 mm
- net GPA1: track 93.4 -> 89.9 mm
- net GPB0: track 57.1 -> 53.7 mm
- net GPA2: track 75.6 -> 72.2 mm
- net I2C_SDA: track 130.0 -> 127.1 mm
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Other:
- outline, holes or cut-outs redrawn
- board text added: "PCB-E21-TVS, v03-16"
- board text removed: "PCB-E21-TVS, v02-16"
