File: PCBs/PCB-ENCODER2a/PCB-ENCODER2a.brd (EAGLE design)
At the start: 27.9 x 35.6 mm, 21 parts, among them IC1 MCP23017SS, IC2 74HCT14D, SW1 EC12E_SW, SW2 EC12E_SW

Commit message: PCBS updated
Parts:
- C1: value 10uF -> 22uF
- C2, C5: value 100nF -> 10nF
- R13, R2: value 10K -> 0R
- R3, R4: value 10K -> 100K
Changed lines of the file:
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@@
 <setting verticaltext="up"/>
 </settings>
-<grid distance="1" unitdist="mm" unit="mm" style="lines" multiple="1" display="yes" altdistance="10" altunitdist="mil" altunit="mil"/>
+<grid distance="1" unitdist="mm" unit="mil" style="lines" multiple="1" display="yes" altdistance="10" altunitdist="mil" altunit="mil"/>
 <layers>
 <layer number="1" name="Top" color="4" fill="1" visible="yes" active="yes"/>
@@
 <attribute name="MF" value="" x="35.56" y="15.24" size="1.778" layer="27" display="off"/>
 <attribute name="OC_FARNELL" value="1520813" x="35.56" y="15.24" size="1.778" layer="27" display="off"/>
-<attribute name="NAME" x="15.615" y="27.475" size="1.27" layer="25" rot="R180"/>
+<attribute name="NAME" x="15.107" y="27.729" size="0.7112" layer="25" rot="R180"/>
 <attribute name="VALUE" x="18.74" y="22.75" size="1.27" layer="27" rot="R180"/>
 </element>
-<element name="C1" library="SparkFun" package="0805" value="10uF" x="23.76" y="10.129" smashed="yes" rot="MR0">
+<element name="C1" library="SparkFun" package="0805" value="22uF" x="23.76" y="10.129" smashed="yes" rot="MR0">
 <attribute name="NAME" x="24.649" y="10.891" size="0.6096" layer="26" font="vector" rot="MR0"/>
 <attribute name="VALUE" x="24.776" y="8.986" size="0.4064" layer="28" font="vector" rot="MR0"/>
 </element>
-<element name="C2" library="SparkFun" package="0603-CAP" value="100nF" x="21.847" y="23.843" rot="MR180"/>
-<element name="C3" library="SparkFun" package="0603-CAP" value="10nF" x="12.713" y="20.91" rot="MR180"/>
-<element name="C4" library="SparkFun" package="0603-CAP" value="10nF" x="14.017" y="33.637" rot="MR0"/>
-<element name="R2" library="SparkFun" package="0603-RES" value="10K" x="20.127" y="20.287" rot="MR270"/>
+<element name="C2" library="SparkFun" package="0603-CAP" value="10nF" x="21.847" y="23.843" smashed="yes" rot="MR180">
+<attribute name="NAME" x="20.958" y="23.081" size="0.7112" layer="26" font="vector" rot="MR180"/>
+<attribute name="VALUE" x="20.831" y="24.986" size="0.4064" layer="28" font="vector" rot="MR180"/>
+</element>
+<element name="C3" library="SparkFun" package="0603-CAP" value="10nF" x="12.713" y="20.91" smashed="yes" rot="MR180">
+<attribute name="NAME" x="14.11" y="21.164" size="0.7112" layer="26" font="vector" rot="MR180"/>
+<attribute name="VALUE" x="11.697" y="22.053" size="0.4064" layer="28" font="vector" rot="MR180"/>
+</element>
+<element name="C4" library="SparkFun" package="0603-CAP" value="10nF" x="14.017" y="33.637" smashed="yes" rot="MR0">
+<attribute name="NAME" x="14.398" y="34.399" size="0.7112" layer="26" font="vector" rot="MR0"/>
+<attribute name="VALUE" x="15.033" y="32.494" size="0.4064" layer="28" font="vector" rot="MR0"/>
+</element>
+<element name="R2" library="SparkFun" package="0603-RES" value="0R" x="20.127" y="20.287" smashed="yes" rot="MR270">
+<attribute name="NAME" x="20.381" y="18.89" size="0.7112" layer="26" font="vector" rot="MR270"/>
+<attribute name="VALUE" x="21.27" y="21.303" size="0.4064" layer="28" font="vector" rot="MR270"/>
+</element>
 <element name="U$20" library="SKAARHOJ" package="3.2MMPAD6MM" value="GNDPAD6MM" x="3.5" y="3.5"/>
 <element name="U$21" library="SKAARHOJ" package="3.2MMPAD6MM" value="GNDPAD6MM" x="24.44" y="32.06"/>
@@
 <attribute name="MF" value="" x="-3.81" y="31.75" size="1.778" layer="27" display="off"/>
 <attribute name="OC_FARNELL" value="1520813" x="-3.81" y="31.75" size="1.778" layer="27" display="off"/>
-<attribute name="NAME" x="12.74" y="8.5" size="1.27" layer="25"/>
+<attribute name="NAME" x="12.74" y="9.262" size="0.7112" layer="25"/>
 <attribute name="VALUE" x="17.47" y="-0.11" size="1.27" layer="27" rot="R180"/>
 </element>
-<element name="C5" library="SparkFun" package="0603-CAP" value="100nF" x="12.702" y="4.54" rot="MR270"/>
-<element name="C6" library="SparkFun" package="0603-CAP" value="10nF" x="10.922" y="4.556" rot="MR90"/>
-<element name="C7" library="SparkFun" package="0603-CAP" value="10nF" x="13.97" y="16.24" rot="MR0"/>
-<element name="R13" library="SparkFun" package="0603-RES" value="10K" x="14.7" y="4.492" rot="MR270"/>
-<element name="IC1" library="microchip" package="SSOP28" value="MCP23017SS" x="5.5" y="16.08" rot="MR270">
+<element name="C5" library="SparkFun" package="0603-CAP" value="10nF" x="12.702" y="4.54" smashed="yes" rot="MR270">
+<attribute name="NAME" x="12.956" y="7.461" size="0.7112" layer="26" font="vector" rot="MR270"/>
+<attribute name="VALUE" x="13.845" y="5.556" size="0.4064" layer="28" font="vector" rot="MR270"/>
+</element>
+<element name="C6" library="SparkFun" package="0603-CAP" value="10nF" x="10.922" y="4.556" smashed="yes" rot="MR90">
+<attribute name="NAME" x="10.716" y="6.191" size="0.7112" layer="26" font="vector" rot="MR90"/>
+<attribute name="VALUE" x="9.779" y="3.54" size="0.4064" layer="28" font="vector" rot="MR90"/>
+</element>
+<element name="C7" library="SparkFun" package="0603-CAP" value="10nF" x="13.97" y="16.24" smashed="yes" rot="MR0">
+<attribute name="NAME" x="14.351" y="17.002" size="0.7112" layer="26" font="vector" rot="MR0"/>
+<attribute name="VALUE" x="14.986" y="15.097" size="0.4064" layer="28" font="vector" rot="MR0"/>
+</element>
+<element name="R13" library="SparkFun" package="0603-RES" value="0R" x="14.7" y="4.492" smashed="yes" rot="MR270">
+<attribute name="NAME" x="14.954" y="8.175" size="0.7112" layer="26" font="vector" rot="MR270"/>
+<attribute name="VALUE" x="15.843" y="5.508" size="0.4064" layer="28" font="vector" rot="MR270"/>
+</element>
+<element name="IC1" library="microchip" package="SSOP28" value="MCP23017SS" x="5.5" y="16.08" smashed="yes" rot="MR270">
 <attribute name="OC_NEWARK" value="31K2960" x="5.5" y="16.08" size="1.778" layer="28" rot="MR270" display="off"/>
 <attribute name="MPN" value="MCP23017-E/SS" x="5.5" y="16.08" size="1.778" layer="28" rot="MR270" display="off"/>
 <attribute name="MF" value="MICROCHIP" x="5.5" y="16.08" size="1.778" layer="28" rot="MR270" display="off"/>
 <attribute name="OC_FARNELL" value="1467674" x="5.5" y="16.08" size="1.778" layer="28" rot="MR270" display="off"/>
-</element>
-<element name="C14" library="SparkFun" package="0603-CAP" value="100nF" x="11.828" y="13.864" rot="MR0"/>
+<attribute name="NAME" x="7.1139" y="21.556" size="0.7112" layer="26" rot="MR0"/>
+<attribute name="VALUE" x="6.18" y="19.9799" size="1.27" layer="28" rot="MR270"/>
+</element>
+<element name="C14" library="SparkFun" package="0603-CAP" value="100nF" x="11.828" y="13.864" smashed="yes" rot="MR0">
+<attribute name="NAME" x="12.717" y="12.594" size="0.7112" layer="26" font="vector" rot="MR0"/>
+<attribute name="VALUE" x="12.844" y="12.721" size="0.4064" layer="28" font="vector" rot="MR0"/>
+</element>
 <element name="U$19" library="SKAARHOJ" package="3BITADDR" value="3BITADDR" x="4.532" y="31.732" rot="MR0"/>
-<element name="IC2" library="74xx-eu" package="SO14" value="74HCT14D" x="14.036" y="26.398" rot="MR270"/>
-<element name="C18" library="SparkFun" package="0603-CAP" value="100nF" x="11.222" y="32.07" rot="MR180"/>
-<element name="R3" library="SparkFun" package="0603-RES" value="10K" x="18.354" y="20.27" rot="MR90"/>
-<element name="R4" library="SparkFun" package="0603-RES" value="10K" x="16.414" y="4.384" rot="MR90"/>
+<element name="IC2" library="74xx-eu" package="SO14" value="74HCT14D" x="14.036" y="26.398" smashed="yes" rot="MR270">
+<attribute name="VALUE" x="14.798" y="29.573" size="1.27" layer="28" ratio="10" rot="MR270"/>
+<attribute name="NAME" x="17.973" y="30.97" size="0.7112" layer="26" ratio="10" rot="MR0"/>
+</element>
+<element name="C18" library="SparkFun" package="0603-CAP" value="100nF" x="11.222" y="32.07" smashed="yes" rot="MR180">
+<attribute name="NAME" x="12.873" y="32.324" size="0.7112" layer="26" font="vector" rot="MR180"/>
+<attribute name="VALUE" x="10.206" y="33.213" size="0.4064" layer="28" font="vector" rot="MR180"/>
+</element>
+<element name="R3" library="SparkFun" package="0603-RES" value="100K" x="18.354" y="20.27" smashed="yes" rot="MR90">
+<attribute name="NAME" x="18.148" y="17.603" size="0.7112" layer="26" font="vector" rot="MR90"/>
+<attribute name="VALUE" x="17.211" y="19.254" size="0.4064" layer="28" font="vector" rot="MR90"/>
+</element>
+<element name="R4" library="SparkFun" package="0603-RES" value="100K" x="16.414" y="4.384" smashed="yes" rot="MR90">
+<attribute name="NAME" x="16.16" y="6.035" size="0.7112" layer="26" font="vector" rot="MR90"/>
+<attribute name="VALUE" x="15.271" y="3.368" size="0.4064" layer="28" font="vector" rot="MR90"/>
+</element>
 </elements>
 <signals>

Commit message: asdf
Parts:
- removed R13, R2: 0R, SparkFun:0603-RES
Connections:
- removed net N$124: C2.1, IC2.13, R2.1
- removed net N$125: C5.1, IC2.9, R13.1
- net N$1: now also C2.1, IC2.13; no longer R2.2
- net N$6: now also C5.1, IC2.9; no longer R13.2
Routing:
- net N$6: track 3.94 -> 35.2 mm, vias 0 -> 2
- net N$125: track 22.8 -> 0.00 mm, vias 2 -> 0
- net N$1: track 3.87 -> 23.5 mm, vias 0 -> 2
- net N$124: track 14.9 -> 0.00 mm, vias 2 -> 0
Other:
- board text added: "PCB-ENCODER2 v04-15"
- board text added: "SKAARHOJ 2015"
- board text removed: "PCB-ENCODER2 v10-14"
- board text removed: "SKAARHOJ 2014"
Changed lines of the file:
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@@
 <?xml version="1.0" encoding="utf-8"?>
 <!DOCTYPE eagle SYSTEM "eagle.dtd">
-<eagle version="7.1.0">
+<eagle version="7.2.0">
 <drawing>
 <settings>
@@
 <wire x1="27.94" y1="35.56" x2="0" y2="35.56" width="0" layer="20"/>
 <wire x1="0" y1="35.56" x2="0" y2="0" width="0" layer="20"/>
-<text x="27.575" y="12.573" size="1.016" layer="122" rot="MR270">SKAARHOJ 2014</text>
+<text x="27.575" y="12.573" size="1.016" layer="122" rot="MR270">SKAARHOJ 2015</text>
 <rectangle x1="4.915775" y1="8.815921875" x2="6.77759375" y2="8.900759375" layer="200" rot="R90"/>
 <rectangle x1="5.592684375" y1="10.76283125" x2="6.100684375" y2="10.84766875" layer="200" rot="R90"/>
@@
 <wire x1="21" y1="12" x2="21" y2="15" width="0.4064" layer="122"/>
 <wire x1="21" y1="15" x2="24" y2="15" width="0.4064" layer="122"/>
-<text x="0.254" y="6.858" size="0.8128" layer="122" rot="MR90">PCB-ENCODER2 v10-14</text>
+<text x="0.254" y="6.858" size="0.8128" layer="122" rot="MR90">PCB-ENCODER2 v04-15</text>
 </plain>
 <attributes>
@@
 <attribute name="VALUE" x="15.033" y="32.494" size="0.4064" layer="28" font="vector" rot="MR0"/>
 </element>
-<element name="R2" library="SparkFun" package="0603-RES" value="0R" x="20.127" y="20.287" smashed="yes" rot="MR270">
-<attribute name="NAME" x="20.381" y="18.89" size="0.7112" layer="26" font="vector" rot="MR270"/>
-<attribute name="VALUE" x="21.27" y="21.303" size="0.4064" layer="28" font="vector" rot="MR270"/>
-</element>
 <element name="U$20" library="SKAARHOJ" package="3.2MMPAD6MM" value="GNDPAD6MM" x="3.5" y="3.5"/>
 <element name="U$21" library="SKAARHOJ" package="3.2MMPAD6MM" value="GNDPAD6MM" x="24.44" y="32.06"/>
@@
 <attribute name="NAME" x="14.351" y="17.002" size="0.7112" layer="26" font="vector" rot="MR0"/>
 <attribute name="VALUE" x="14.986" y="15.097" size="0.4064" layer="28" font="vector" rot="MR0"/>
-</element>
-<element name="R13" library="SparkFun" package="0603-RES" value="0R" x="14.7" y="4.492" smashed="yes" rot="MR270">
-<attribute name="NAME" x="14.954" y="8.175" size="0.7112" layer="26" font="vector" rot="MR270"/>
-<attribute name="VALUE" x="15.843" y="5.508" size="0.4064" layer="28" font="vector" rot="MR270"/>
 </element>
 <element name="IC1" library="microchip" package="SSOP28" value="MCP23017SS" x="5.5" y="16.08" smashed="yes" rot="MR270">
@@
 <signal name="N$1">
 <contactref element="SW1" pad="B"/>
-<contactref element="R2" pad="2"/>
 <contactref element="R3" pad="1"/>
 <wire x1="20.1168" y1="19.5072" x2="18.3896" y2="19.5072" width="0.2032" layer="16"/>
 <wire x1="18.3896" y1="19.5072" x2="18.354" y2="19.42" width="0.2032" layer="16"/>
-<wire x1="20.1168" y1="19.5072" x2="20.127" y2="19.437" width="0.2032" layer="16"/>
 <wire x1="16.764" y1="19.4056" x2="18.288" y2="19.4056" width="0.2032" layer="16"/>
 <wire x1="16.5608" y1="19.2024" x2="16.764" y2="19.4056" width="0.2032" layer="16"/>
 <wire x1="18.288" y1="19.4056" x2="18.354" y2="19.42" width="0.2032" layer="16"/>
 <wire x1="16.5608" y1="19.2024" x2="16.47" y2="19.17" width="0.2032" layer="16"/>
+<contactref element="IC2" pad="13"/>
+<contactref element="C2" pad="1"/>
+<wire x1="20.955" y1="19.685" x2="20.955" y2="22.86" width="0.2032" layer="16"/>
+<wire x1="20.955" y1="22.86" x2="20.955" y2="23.495" width="0.2032" layer="16"/>
+<wire x1="18.415" y1="19.685" x2="20.955" y2="19.685" width="0.2032" layer="16"/>
+<wire x1="20.955" y1="23.495" x2="20.997" y2="23.843" width="0.2032" layer="16"/>
+<wire x1="18.415" y1="19.685" x2="18.354" y2="19.42" width="0.2032" layer="16"/>
+<wire x1="12.065" y1="28.575" x2="11.43" y2="29.21" width="0.2032" layer="16"/>
+<wire x1="13.335" y1="28.575" x2="12.065" y2="28.575" width="0.2032" layer="16"/>
+<wire x1="19.05" y1="22.86" x2="13.335" y2="28.575" width="0.2032" layer="1"/>
+<wire x1="20.955" y1="22.86" x2="19.05" y2="22.86" width="0.2032" layer="16"/>
+<wire x1="11.43" y1="29.21" x2="10.9626" y2="28.938" width="0.2032" layer="16"/>
+<via x="13.335" y="28.575" extent="1-16" drill="0.4064"/>
+<via x="19.05" y="22.86" extent="1-16" drill="0.4064"/>
 </signal>
 <signal name="I2C_SDA">
@@
 <signal name="N$6">
 <contactref element="SW2" pad="B"/>
-<contactref element="R13" pad="2"/>
 <contactref element="R4" pad="1"/>
 <wire x1="16.3576" y1="3.556" x2="14.732" y2="3.556" width="0.2032" layer="16"/>
-<wire x1="14.732" y1="3.556" x2="14.7" y2="3.642" width="0.2032" layer="16"/>
 <wire x1="16.3576" y1="3.556" x2="16.414" y2="3.534" width="0.2032" layer="16"/>
 <wire x1="16.4592" y1="1.4224" x2="16.4592" y2="3.4544" width="0.2032" layer="16"/>
 <wire x1="16.4592" y1="3.4544" x2="16.414" y2="3.534" width="0.2032" layer="16"/>
 <wire x1="16.4592" y1="1.4224" x2="16.47" y2="1.39" width="0.2032" layer="16"/>
+<contactref element="C5" pad="1"/>
+<contactref element="IC2" pad="9"/>
+<wire x1="14.605" y1="5.08" x2="12.7" y2="5.08" width="0.2032" layer="16"/>
+<wire x1="15.875" y1="3.81" x2="14.605" y2="5.08" width="0.2032" layer="16"/>
+<wire x1="16.51" y1="3.81" x2="15.875" y2="3.81" width="0.2032" layer="16"/>
+<wire x1="12.7" y1="5.08" x2="12.702" y2="5.39" width="0.2032" layer="16"/>
+<wire x1="16.51" y1="3.81" x2="16.414" y2="3.534" width="0.2032" layer="16"/>
+<wire x1="13.335" y1="24.13" x2="11.43" y2="24.13" width="0.2032" layer="16"/>
+<wire x1="14.605" y1="24.13" x2="13.335" y2="24.13" width="0.2032" layer="1"/>
+<wire x1="18.415" y1="20.32" x2="14.605" y2="24.13" width="0.2032" layer="1"/>
+<wire x1="18.415" y1="12.065" x2="18.415" y2="20.32" width="0.2032" layer="1"/>
+<wire x1="16.51" y1="10.16" x2="18.415" y2="12.065" width="0.2032" layer="1"/>
+<wire x1="12.7" y1="6.35" x2="16.51" y2="10.16" width="0.2032" layer="16"/>
+<wire x1="12.7" y1="5.715" x2="12.7" y2="6.35" width="0.2032" layer="16"/>
+<wire x1="11.43" y1="24.13" x2="10.9626" y2="23.858" width="0.2032" layer="16"/>
+<wire x1="12.7" y1="5.715" x2="12.702" y2="5.39" width="0.2032" layer="16"/>
+<via x="13.335" y="24.13" extent="1-16" drill="0.4064"/>
+<via x="16.51" y="10.16" extent="1-16" drill="0.4064"/>
 </signal>
 <signal name="A0">
@@
 <wire x1="2.2352" y1="31.6992" x2="2.332" y2="31.732" width="0.2032" layer="16"/>
 </signal>
-<signal name="N$124">
-<contactref element="C2" pad="1"/>
-<contactref element="R2" pad="1"/>
-<contactref element="IC2" pad="13"/>
-<wire x1="20.2184" y1="23.0632" x2="20.2184" y2="21.2344" width="0.2032" layer="16"/>
-<wire x1="20.9296" y1="23.7744" x2="20.3708" y2="23.2156" width="0.2032" layer="16"/>
-<wire x1="20.3708" y1="23.2156" x2="20.2184" y2="23.0632" width="0.2032" layer="16"/>
-<wire x1="20.2184" y1="21.2344" x2="20.127" y2="21.137" width="0.2032" layer="16"/>
-<wire x1="20.9296" y1="23.7744" x2="20.997" y2="23.843" width="0.2032" layer="16"/>
-<wire x1="14.224" y1="28.8544" x2="10.9728" y2="28.8544" width="0.2032" layer="16"/>
-<wire x1="19.812" y1="23.2664" x2="14.224" y2="28.8544" width="0.2032" layer="1"/>
-<wire x1="20.32" y1="23.2664" x2="19.812" y2="23.2664" width="0.2032" layer="16"/>
-<wire x1="10.9728" y1="28.8544" x2="10.9626" y2="28.938" width="0.2032" layer="16"/>
-<wire x1="20.32" y1="23.2664" x2="20.3708" y2="23.2156" width="0.2032" layer="16"/>
-<via x="14.224" y="28.8544" extent="1-16" drill="0.4064"/>
-<via x="19.812" y="23.2664" extent="1-16" drill="0.4064"/>
-</signal>
-<signal name="N$125">
-<contactref element="C5" pad="1"/>
-<contactref element="R13" pad="1"/>
-<contactref element="IC2" pad="9"/>
-<wire x1="12.8016" y1="5.3848" x2="14.6304" y2="5.3848" width="0.2032" layer="16"/>
-<wire x1="14.6304" y1="5.3848" x2="14.7" y2="5.342" width="0.2032" layer="16"/>
-<wire x1="12.8016" y1="5.3848" x2="12.702" y2="5.39" width="0.2032" layer="16"/>
-<wire x1="14.6304" y1="10.3632" x2="14.6304" y2="5.4864" width="0.2032" layer="16"/>
-<wire x1="14.732" y1="10.4648" x2="14.6304" y2="10.3632" width="0.2032" layer="16"/>
-<wire x1="14.732" y1="17.8816" x2="14.732" y2="10.4648" width="0.2032" layer="1"/>
-<wire x1="15.1384" y1="18.288" x2="14.732" y2="17.8816" width="0.2032" layer="1"/>
-<wire x1="15.1384" y1="20.2184" x2="15.1384" y2="18.288" width="0.2032" layer="1"/>
-<wire x1="12.7" y1="22.6568" x2="15.1384" y2="20.2184" width="0.2032" layer="1"/>
-<wire x1="11.5824" y1="23.7744" x2="12.7" y2="22.6568" width="0.2032" layer="16"/>
-<wire x1="10.9728" y1="23.7744" x2="11.5824" y2="23.7744" width="0.2032" layer="16"/>
-<wire x1="14.6304" y1="5.4864" x2="14.7" y2="5.342" width="0.2032" layer="16"/>
-<wire x1="10.9728" y1="23.7744" x2="10.9626" y2="23.858" width="0.2032" layer="16"/>
-<via x="14.732" y="10.4648" extent="1-16" drill="0.4064"/>
-<via x="12.7" y="22.6568" extent="1-16" drill="0.4064"/>
-</signal>
 </signals>
