File: PCBs/PCB-ETHMG-BOS/PCB-ETHMG-BOS.brd (EAGLE design)
At the start: 100 x 69 mm, 48 parts, among them U1 ARDUINO-MEGAFULL

Commit message: PCBS updated
Parts:
- removed CONFA: (no value), SKAARHOJ:PUSHBUTTON
- moved L3 23.5 mm to (37.0, 67.0), turned to 0 degrees
- moved CONF 19.0 mm to (9.40, 53.3)
- moved RESET 19.0 mm to (11.9, 45.0)
- moved RESETA 19.0 mm to (9.40, 45.0)
- moved L6 7.07 mm to (66.0, 4.00)
- moved R1 5.66 mm to (62.0, 63.0)
- moved R2 5.66 mm to (66.0, 63.0)
- moved C1 4.12 mm to (62.0, 66.0)
- moved C2 4.12 mm to (66.0, 66.0)
- moved L1 3.62 mm to (84.7, 34.5), turned to 0 degrees
- moved L2 1.00 mm to (81.0, 62.0), turned to 0 degrees
- moved L4 1.00 mm to (37.0, 64.0), turned to 0 degrees
- moved C6 0.61 mm to (36.6, 1.30)
- moved C3 0.44 mm to (36.6, 3.43)
Connections:
- net D37: no longer CONFA.3
- net GND: no longer CONFA.1
Routing:
- net N$2: track 2.64 -> 84.5 mm, vias 0 -> 2
- net D37: track 94.0 -> 144.4 mm, vias 0 -> 3
- net GPIO3-1: track 76.3 -> 34.3 mm, vias 4 -> 1
- net GND: track 419.9 -> 456.6 mm, vias 14 -> 5
- net N$7: track 80.5 -> 107.9 mm, vias 4 -> 5
- net 5V: track 257.9 -> 280.6 mm, vias 7 -> 6
- net RESET: track 26.5 -> 47.6 mm
- net D23: track 125.0 -> 104.0 mm, vias 4 -> 3
- net N$11: track 81.7 -> 61.1 mm, vias 0 -> 4
- net D22: track 121.5 -> 101.9 mm, vias 3 -> 4
- net A7: track 56.5 -> 71.9 mm, vias 3 -> 1
- net A9: track 52.5 -> 67.1 mm
- net A1: track 41.9 -> 54.0 mm
- net A5: track 59.8 -> 48.4 mm, vias 3 -> 1
- net A0: track 109.9 -> 121.1 mm, vias 4 -> 3
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Other:
- outline, holes or cut-outs redrawn
- board text added: "SKAARHOJ 2013"
- board text added: "v07-13"
- board text removed: "SKAARHOJ 2014"
- board text removed: "v10-14"

Commit message: asfd
Other:
- board text added: "PCB-ETHMG-BOS"
- board text added: "SKAARHOJ 2015"
- board text added: "v08-15"
- board text removed: "PCB-ARD-MMBOS"
- board text removed: "SKAARHOJ 2013"
- board text removed: "v07-13"
Changed lines of the file:
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@@
 <?xml version="1.0" encoding="utf-8"?>
 <!DOCTYPE eagle SYSTEM "eagle.dtd">
-<eagle version="7.1.0">
+<eagle version="7.3.0">
 <drawing>
 <settings>
@@
 <plain>
 <text x="29.718" y="63.9285" size="1.778" layer="121" font="vector" align="center">SKAARHOJ
-2013</text>
+2015</text>
 <wire x1="71.12" y1="50.657" x2="73.4695" y2="50.657" width="0.4064" layer="121"/>
 <wire x1="73.4695" y1="50.657" x2="73.4695" y2="50.5935" width="0.4064" layer="121"/>
@@
 <wire x1="92.075" y1="1" x2="92.075" y2="4.175" width="0.4064" layer="121"/>
 <wire x1="92.075" y1="4.175" x2="95.25" y2="4.175" width="0.4064" layer="121"/>
-<text x="13.97" y="67.04" size="1.016" layer="121">PCB-ARD-MMBOS</text>
-<text x="13.97" y="65.77" size="0.8128" layer="121">v07-13</text>
+<text x="13.97" y="67.04" size="1.016" layer="121">PCB-ETHMG-BOS</text>
+<text x="13.97" y="65.77" size="0.8128" layer="121">v08-15</text>
 <text x="89.535" y="61.96" size="0.8128" layer="121">5V</text>
 <text x="96.52" y="61.96" size="0.8128" layer="121">GND</text>
