File: PCBs/PCB-SDB-1x4/PCB-SDB-1x4.brd (EAGLE design)
At the start: 108 x 23 mm, 13 parts, among them IC1 MCP23017SS

Commit message: PCBS updated
Parts:
- added C10, C12, C2, C4, C7: 100nF, SparkFun:0603-CAP
- added C9: 22uF, SparkFun:0805
- added L4: ILHB0805ER121V, SparkFun:0805
- C3: value 10uF -> 100nF; device SparkFun:0805 -> SparkFun:0603-CAP
- moved C3 66.2 mm to (94.6, 3.81), turned to 0 degrees
Connections:
- new net ARD_5V: C12.1, L4.1, SERIAL.2
- net 5V: now also C10.1, C2.1, C4.1, C7.1, C9.1, L4.2; no longer SERIAL.2
- net GND: now also C10.2, C12.2, C2.2, C4.2, C7.2, C9.2
Routing:
- net GND: track 248.8 -> 279.7 mm, vias 0 -> 1
- net SDI_SCLK: track 104.2 -> 80.9 mm
- net 5V: track 129.9 -> 151.4 mm
- net A2: track 39.9 -> 30.1 mm, vias 1 -> 4
- net A1: track 35.1 -> 30.7 mm, vias 1 -> 3
- net ARD_5V: track 0.00 -> 4.07 mm
- net SDI_MOSI: track 82.0 -> 85.9 mm, vias 0 -> 1
- net A0: track 29.5 -> 31.8 mm, vias 1 -> 2
- net GPB3: track 41.6 -> 39.6 mm, vias 1 -> 0
- net GPB0: track 41.8 -> 40.1 mm, vias 1 -> 0
- net I2C_SCL: track 33.7 -> 35.1 mm, vias 1 -> 2
- net I2C_SDA: track 30.5 -> 31.1 mm, vias 1 -> 0
- net GPB2: vias 1 -> 0
Other:
- board text added: "SDB-1x4 v10-14"
- board text removed: "SDB-1x4 v06-14"

Commit message: PCB updates
Parts:
- SERIAL: value M04X2 -> M04X2M2X4SMALLER; device SparkFun:2X4 -> SKAARHOJ:M2X4SMALLER
- U$19: value 3BITADDR -> 3BITADDRSMALL; device SKAARHOJ:3BITADDR -> SKAARHOJ:3BITADDR_SMALL
- turned SERIAL to 0 degrees
Connections:
- net 5V: now also U$19.H0; no longer U$19.H3
- net A0: now also U$19.AS0
- net A1: now also U$19.AS1
- net A2: now also U$19.AS2
- net GND: now also U$19.L0; no longer U$19.L3
Routing:
- net GND: track 279.7 -> 261.0 mm
- net GPB3: track 39.6 -> 43.7 mm, vias 0 -> 1
- net SDI_SCLK: track 80.9 -> 81.9 mm
- net 5V: track 151.4 -> 152.4 mm
- net A0: track 31.8 -> 32.5 mm
- net A1: track 30.7 -> 30.1 mm
Other:
- board text added: "SDB-1x4, v02-16"
- board text removed: "SDB-1x4 v10-14"
- board text removed: "SKAARHOJ 2014"
