File: PCBs/PCB-SSB-1x1ENC/PCB-SSB-1x1ENC.brd (EAGLE design)
At the start: 38 x 29.5 mm, 14 parts, among them IC4 MCP23017SS, IC5 74HCT14D, SW1 EC12E_SWCAR1

Commit message: asdf
Parts:
- added SSW1ALT: SMART_SWITCHSMART_SWITCH_8PIN, SKAARHOJ:SMART_SWITCH
- added U$1: 3BITADDRSMALL, SKAARHOJ:3BITADDR_SMALL
- SERIAL: value M04X2 -> M04X2M2X4SMALLER; device SparkFun:2X4 -> SKAARHOJ:M2X4SMALLER
- moved IC5 24.5 mm to (32.6, 24.5), turned to 180 degrees
- moved C3 24.5 mm to (26.5, 22.0), turned to 180 degrees
- moved C9 22.0 mm to (37.1, 4.83)
- moved IC4 21.6 mm to (31.2, 6.10)
- moved C10 20.2 mm to (36.6, 17.9)
- moved C12 18.6 mm to (33.1, 18.9), turned to 0 degrees
- moved C11 15.3 mm to (25.4, 15.2)
- moved R33 10.1 mm to (29.0, 18.9), turned to 0 degrees
- moved C22 5.71 mm to (21.3, 21.6)
- moved SW1 0.49 mm to (31.5, 14.8)
- moved SSW1 0.14 mm to (9.40, 14.8)
- turned SERIAL to 0 degrees
Connections:
- new net AA0: IC4.15, U$1.A0, U$1.AS0
- new net AA1: IC4.16, U$1.A1, U$1.AS1
- new net AA2: IC4.17, U$1.A2, U$1.AS2
- net 5V: now also SSW1ALT.4, U$1.H0, U$1.H1, U$1.H2
- net GND: now also SSW1ALT.1, SSW1ALT.3, U$1.L0, U$1.L1, U$1.L2; no longer IC4.15, IC4.16, IC4.17
- net GPA4S: now also SSW1ALT.2
- net GPB4: now also SSW1ALT.8
- net MOSI: now also SSW1ALT.6
- net SCLK: now also SSW1ALT.7
Routing:
- net AA1: track 0.00 -> 78.8 mm, vias 0 -> 1
- net AD0: track 59.0 -> 9.69 mm, vias 2 -> 1
- net AA2: track 0.00 -> 31.6 mm, vias 0 -> 1
- net GPB4: track 8.10 -> 39.5 mm, vias 1 -> 2
- net AA0: track 0.00 -> 30.7 mm, vias 0 -> 1
- net D3: track 40.7 -> 11.5 mm, vias 2 -> 0
- net GND: track 113.4 -> 141.9 mm
- net 5V: track 53.1 -> 80.9 mm
- net GPA4S: track 11.7 -> 34.3 mm, vias 0 -> 1
- net N$33: track 32.2 -> 14.3 mm, vias 2 -> 0
- net SCLK: track 6.72 -> 23.9 mm
- net MOSI: track 6.89 -> 16.0 mm
- net D2: track 21.4 -> 17.7 mm
- net I2C_SCL: track 20.4 -> 23.0 mm
- net I2C_SDA: track 23.3 -> 21.8 mm, vias 1 -> 2
Other:
- board text added: "PCB-SSB-1x1ENC, v02-16b SKAARHOJ"
- board text removed: "PCB-SSB-1x1ENC, v02-16 SKAARHOJ"

Commit message: Updates
Parts:
- moved C22 12.7 mm to (21.8, 8.89), turned to 0 degrees
- turned SERIAL to 180 degrees
Routing:
- net AA1: track 78.8 -> 30.7 mm, vias 1 -> 3
- net AA0: track 30.7 -> 72.1 mm
- net I2C_SDA: track 21.8 -> 39.4 mm
- net 5V: track 80.9 -> 96.7 mm, vias 1 -> 3
- net I2C_SCL: track 23.0 -> 35.4 mm, vias 1 -> 2
- net GPB4: track 39.5 -> 31.3 mm
- net MOSI: track 16.0 -> 22.6 mm
- net SCLK: track 23.9 -> 28.4 mm
- net GPA4S: track 34.3 -> 38.1 mm
- net AA2: track 31.6 -> 34.8 mm
- net GND: track 141.9 -> 143.5 mm
Other:
- board text added: "PCB-SSB-1x1ENC, v03-16 SKAARHOJ"
- board text removed: "PCB-SSB-1x1ENC, v02-16b SKAARHOJ"
