File: PCBs/PCB-SSB-1x2b/PCB-SSB-1x2b.brd (EAGLE design)
At the start: 54.5 x 18 mm, 9 parts, among them IC1 MCP23017SS

Commit message: Updated boards
Updated boards with logo before first sending to Alma.
Routing:
- added copper zone on layer 1, net GND
- added copper zone on layer 16, net GND
Other:
- board text added: "v07-13"
- board text removed: "v13-05-13"

Commit message: PCBS updated
Parts:
- removed C3: 10uF, SparkFun:0805
- added C10, C12, C2, C7: 100nF, SparkFun:0603-CAP
- added C9: 22uF, SparkFun:0805
- added L4: ILHB0805ER121V, SparkFun:0805
- added PC2: 47u, rcl:PANASONIC_D
Connections:
- new net ARD_5V: C12.1, L4.1, SERIAL.2
- net 5V: now also C10.1, C2.1, C7.1, C9.1, L4.2, PC2.+; no longer C3.1, SERIAL.2
- net GND: now also C10.2, C12.2, C2.2, C7.2, C9.2, PC2.-; no longer C3.2
Routing:
- net GND: track 80.1 -> 116.5 mm, vias 1 -> 4
- net 5V: track 57.1 -> 80.8 mm, vias 0 -> 4
- net SDI_SCLK: track 27.8 -> 45.9 mm
- net A2: track 8.47 -> 20.1 mm
- net ARD_5V: track 0.00 -> 10.1 mm, vias 0 -> 1
- net I2C_SDA: track 27.9 -> 25.5 mm, vias 2 -> 0
- net GPA1: track 34.6 -> 33.6 mm
- net I2C_SCL: track 24.6 -> 25.3 mm
- net A1: track 7.52 -> 8.13 mm, vias 1 -> 0
- net SDI_MOSI: track 33.4 -> 33.2 mm, vias 3 -> 0
- net GPA0: track 13.0 -> 12.8 mm, vias 1 -> 0
- net GPB1: vias 1 -> 0
- net A0: vias 1 -> 0
Other:
- board text added: "SKAARHOJ 2014"
- board text added: "v10-14"
- board text removed: "SKAARHOJ 2013"
- board text removed: "v07-13"
