File: PCBs/PCB-DISPLAYDOGM2/PCB-DISPLAYDOGM2.sch (EAGLE design)
At the start: 34 parts, among them IC1 MCP23017SS, IC2 74HC14D, SW1 EC12E_SW, SW2 EC12E_SW

Commit message: asdf
Parts:
- renumbered U$3 to DISP
Changed lines of the file:
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@@
 <part name="U$2" library="SKAARHOJ" deviceset="GNDPAD" device="6MM" value="GNDPAD6MM"/>
 <part name="U$20" library="SKAARHOJ" deviceset="GNDPAD" device="6MM" value="GNDPAD6MM"/>
-<part name="U$3" library="SKAARHOJ" deviceset="DOGM_DISPLAY" device=""/>
+<part name="DISP" library="SKAARHOJ" deviceset="DOGM_DISPLAY" device=""/>
 <part name="R1" library="SparkFun" deviceset="RESISTOR" device="0603-RES" value="30R/0.1W"/>
 <part name="R3" library="SparkFun" deviceset="RESISTOR" device="0603-RES" value="30R/0.1W"/>
@@
 <instance part="U$2" gate="G$1" x="175.26" y="5.08"/>
 <instance part="U$20" gate="G$1" x="175.26" y="-7.62"/>
-<instance part="U$3" gate="G$1" x="-38.1" y="-43.18"/>
+<instance part="DISP" gate="G$1" x="-38.1" y="-43.18"/>
 <instance part="R1" gate="G$1" x="-43.18" y="-15.24" rot="R90"/>
 <instance part="R3" gate="G$1" x="-33.02" y="-15.24" rot="R90"/>
@@
 </segment>
 <segment>
-<pinref part="U$3" gate="G$1" pin="VIN"/>
+<pinref part="DISP" gate="G$1" pin="VIN"/>
 <wire x1="-58.42" y1="-55.88" x2="-60.96" y2="-55.88" width="0.1524" layer="91"/>
-<pinref part="U$3" gate="G$1" pin="VOUT"/>
+<pinref part="DISP" gate="G$1" pin="VOUT"/>
 <wire x1="-58.42" y1="-58.42" x2="-60.96" y2="-58.42" width="0.1524" layer="91"/>
 <wire x1="-60.96" y1="-58.42" x2="-60.96" y2="-55.88" width="0.1524" layer="91"/>
-<pinref part="U$3" gate="G$1" pin="VDD"/>
+<pinref part="DISP" gate="G$1" pin="VDD"/>
 <wire x1="-58.42" y1="-40.64" x2="-60.96" y2="-40.64" width="0.1524" layer="91"/>
 <wire x1="-60.96" y1="-55.88" x2="-60.96" y2="-40.64" width="0.1524" layer="91"/>
@@
 </segment>
 <segment>
-<pinref part="U$3" gate="G$1" pin="RESET_"/>
+<pinref part="DISP" gate="G$1" pin="RESET_"/>
 <wire x1="-15.24" y1="-53.34" x2="-12.7" y2="-53.34" width="0.1524" layer="91"/>
 <label x="-12.7" y="-53.34" size="1.778" layer="95"/>
 </segment>
 <segment>
-<pinref part="U$3" gate="G$1" pin="D5"/>
+<pinref part="DISP" gate="G$1" pin="D5"/>
 <wire x1="-48.26" y1="-68.58" x2="-48.26" y2="-71.12" width="0.1524" layer="91"/>
 <wire x1="-48.26" y1="-71.12" x2="-45.72" y2="-71.12" width="0.1524" layer="91"/>
-<pinref part="U$3" gate="G$1" pin="D0"/>
+<pinref part="DISP" gate="G$1" pin="D0"/>
 <wire x1="-45.72" y1="-71.12" x2="-43.18" y2="-71.12" width="0.1524" layer="91"/>
 <wire x1="-43.18" y1="-71.12" x2="-40.64" y2="-71.12" width="0.1524" layer="91"/>
@@
 <wire x1="-38.1" y1="-71.12" x2="-35.56" y2="-71.12" width="0.1524" layer="91"/>
 <wire x1="-35.56" y1="-71.12" x2="-35.56" y2="-68.58" width="0.1524" layer="91"/>
-<pinref part="U$3" gate="G$1" pin="D1"/>
+<pinref part="DISP" gate="G$1" pin="D1"/>
 <wire x1="-38.1" y1="-68.58" x2="-38.1" y2="-71.12" width="0.1524" layer="91"/>
 <junction x="-38.1" y="-71.12"/>
-<pinref part="U$3" gate="G$1" pin="D2"/>
+<pinref part="DISP" gate="G$1" pin="D2"/>
 <wire x1="-40.64" y1="-68.58" x2="-40.64" y2="-71.12" width="0.1524" layer="91"/>
 <junction x="-40.64" y="-71.12"/>
-<pinref part="U$3" gate="G$1" pin="D3"/>
+<pinref part="DISP" gate="G$1" pin="D3"/>
 <wire x1="-43.18" y1="-68.58" x2="-43.18" y2="-71.12" width="0.1524" layer="91"/>
 <junction x="-43.18" y="-71.12"/>
-<pinref part="U$3" gate="G$1" pin="D4"/>
+<pinref part="DISP" gate="G$1" pin="D4"/>
 <wire x1="-45.72" y1="-68.58" x2="-45.72" y2="-71.12" width="0.1524" layer="91"/>
 <junction x="-45.72" y="-71.12"/>
-<pinref part="U$3" gate="G$1" pin="E"/>
+<pinref part="DISP" gate="G$1" pin="E"/>
 <wire x1="-35.56" y1="-71.12" x2="-30.48" y2="-71.12" width="0.1524" layer="91"/>
 <wire x1="-30.48" y1="-71.12" x2="-30.48" y2="-68.58" width="0.1524" layer="91"/>
@@
 </segment>
 <segment>
-<pinref part="U$3" gate="G$1" pin="VSS"/>
+<pinref part="DISP" gate="G$1" pin="VSS"/>
 <wire x1="-58.42" y1="-43.18" x2="-63.5" y2="-43.18" width="0.1524" layer="91"/>
 <label x="-63.5" y="-43.18" size="1.778" layer="95" rot="R180"/>
 </segment>
 <segment>
-<pinref part="U$3" gate="G$1" pin="PSB"/>
+<pinref part="DISP" gate="G$1" pin="PSB"/>
 <wire x1="-15.24" y1="-48.26" x2="-12.7" y2="-48.26" width="0.1524" layer="91"/>
 <label x="-12.7" y="-48.26" size="1.778" layer="95"/>
 </segment>
 <segment>
-<pinref part="U$3" gate="G$1" pin="R/W_"/>
+<pinref part="DISP" gate="G$1" pin="R/W_"/>
 <wire x1="-27.94" y1="-68.58" x2="-27.94" y2="-73.66" width="0.1524" layer="91"/>
 <label x="-27.94" y="-73.66" size="1.778" layer="95" rot="R270"/>
 </segment>
 <segment>
-<pinref part="U$3" gate="G$1" pin="C1/R"/>
+<pinref part="DISP" gate="G$1" pin="C1/R"/>
 <wire x1="-40.64" y1="-35.56" x2="-40.64" y2="-33.02" width="0.1524" layer="91"/>
 <wire x1="-40.64" y1="-33.02" x2="-35.56" y2="-33.02" width="0.1524" layer="91"/>
-<pinref part="U$3" gate="G$1" pin="C2/G"/>
+<pinref part="DISP" gate="G$1" pin="C2/G"/>
 <wire x1="-35.56" y1="-33.02" x2="-35.56" y2="-35.56" width="0.1524" layer="91"/>
 <wire x1="-35.56" y1="-33.02" x2="-30.48" y2="-33.02" width="0.1524" layer="91"/>
@@
 </segment>
 <segment>
-<pinref part="U$3" gate="G$1" pin="D6"/>
+<pinref part="DISP" gate="G$1" pin="D6"/>
 <wire x1="-50.8" y1="-68.58" x2="-50.8" y2="-73.66" width="0.1524" layer="91"/>
 <label x="-50.8" y="-73.66" size="1.778" layer="95" rot="R270"/>
@@
 </segment>
 <segment>
-<pinref part="U$3" gate="G$1" pin="D7"/>
+<pinref part="DISP" gate="G$1" pin="D7"/>
 <wire x1="-53.34" y1="-68.58" x2="-53.34" y2="-73.66" width="0.1524" layer="91"/>
 <label x="-53.34" y="-73.66" size="1.778" layer="95" rot="R270"/>
@@
 </segment>
 <segment>
-<pinref part="U$3" gate="G$1" pin="CSB_"/>
+<pinref part="DISP" gate="G$1" pin="CSB_"/>
 <wire x1="-20.32" y1="-68.58" x2="-20.32" y2="-73.66" width="0.1524" layer="91"/>
 <label x="-20.32" y="-73.66" size="1.778" layer="95" rot="R270"/>
@@
 <net name="C/D" class="0">
 <segment>
-<pinref part="U$3" gate="G$1" pin="RS"/>
+<pinref part="DISP" gate="G$1" pin="RS"/>
 <wire x1="-25.4" y1="-68.58" x2="-25.4" y2="-73.66" width="0.1524" layer="91"/>
 <label x="-25.4" y="-73.66" size="1.778" layer="95" rot="R270"/>
@@
 <segment>
 <pinref part="R1" gate="G$1" pin="1"/>
-<pinref part="U$3" gate="G$1" pin="A1/A"/>
+<pinref part="DISP" gate="G$1" pin="A1/A"/>
 <wire x1="-43.18" y1="-20.32" x2="-43.18" y2="-35.56" width="0.1524" layer="91"/>
 </segment>
@@
 <net name="N$3" class="0">
 <segment>
-<pinref part="U$3" gate="G$1" pin="A2/B"/>
+<pinref part="DISP" gate="G$1" pin="A2/B"/>
 <wire x1="-38.1" y1="-35.56" x2="-38.1" y2="-22.86" width="0.1524" layer="91"/>
 <pinref part="R3" gate="G$1" pin="1"/>

Commit message: PCBS updated
Parts:
- removed C3: 10uF, SparkFun:CAP0805
- added C10, C12: 100nF, SparkFun:CAP0603-CAP
- added C2: 22uF, SparkFun:CAP0805
- added L4: ILHB0805ER121V, SparkFun:INDUCTOR0805
- C4, C7: value 100nF -> 10nF
- R13, R4, R7: value 10K -> 0R
- R5, R6, R8: value 10K -> 100K
Connections:
- new net ARD_5V: C12.1, L4.1, SERIAL.2
- net 5V: now also C10.1, C2.1, L4.2; no longer C3.1, SERIAL.2
- net GND: now also C10.2, C12.2, C2.2; no longer C3.2
Other:
- note removed: "POWER"

Commit message: asdf
Other:
- note added: "Route the SPI_SCLK through schmitt triggers?"
Changed lines of the file:
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@@
 <text x="-99.06" y="-205.74" size="1.778" layer="91">ADR=Bxxx</text>
 <text x="-101.6" y="-218.44" size="3.81" layer="97">CONFIG</text>
+<text x="-106.68" y="-119.38" size="5.08" layer="91">Route the SPI_SCLK through schmitt triggers?</text>
 </plain>
 <instances>

Commit message: asfd
Connections:
- new net N$7: IC2B.O, IC2E.I
- new net N$8: IC2B.I, SERIAL.7
- net GND: no longer IC2B.I, IC2E.I
- net SPI_SCLK: now also IC2E.O; no longer SERIAL.7
Other:
- moved on the sheet: IC2B, IC2E
Changed lines of the file:
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@@
 <instance part="GND4" gate="1" x="200.66" y="-172.72"/>
 <instance part="U$5" gate="G$1" x="200.66" y="-160.02"/>
-<instance part="IC2" gate="B" x="-12.7" y="-251.46"/>
-<instance part="IC2" gate="E" x="-10.16" y="-271.78"/>
+<instance part="IC2" gate="B" x="132.08" y="-104.14"/>
+<instance part="IC2" gate="E" x="157.48" y="-104.14"/>
 <instance part="IC2" gate="F" x="-10.16" y="-287.02"/>
 <instance part="R5" gate="G$1" x="30.48" y="-149.86" rot="R90"/>
@@
 <pinref part="IC2" gate="F" pin="I"/>
 <wire x1="-20.32" y1="-287.02" x2="-30.48" y2="-287.02" width="0.1524" layer="91"/>
-<wire x1="-30.48" y1="-287.02" x2="-30.48" y2="-271.78" width="0.1524" layer="91"/>
-<wire x1="-30.48" y1="-271.78" x2="-30.48" y2="-251.46" width="0.1524" layer="91"/>
-<wire x1="-30.48" y1="-251.46" x2="-30.48" y2="-193.04" width="0.1524" layer="91"/>
+<wire x1="-30.48" y1="-287.02" x2="-30.48" y2="-193.04" width="0.1524" layer="91"/>
 <wire x1="-30.48" y1="-193.04" x2="-12.7" y2="-193.04" width="0.1524" layer="91"/>
 <junction x="-12.7" y="-193.04"/>
-<pinref part="IC2" gate="B" pin="I"/>
-<wire x1="-22.86" y1="-251.46" x2="-30.48" y2="-251.46" width="0.1524" layer="91"/>
-<junction x="-30.48" y="-251.46"/>
-<pinref part="IC2" gate="E" pin="I"/>
-<wire x1="-20.32" y1="-271.78" x2="-30.48" y2="-271.78" width="0.1524" layer="91"/>
-<junction x="-30.48" y="-271.78"/>
 </segment>
 <segment>
@@
 <net name="SPI_SCLK" class="0">
 <segment>
-<pinref part="SERIAL" gate="G$1" pin="7"/>
-<wire x1="129.54" y1="-76.2" x2="119.38" y2="-76.2" width="0.1524" layer="91"/>
-<label x="119.38" y="-76.2" size="1.778" layer="95" rot="R180"/>
-</segment>
-<segment>
 <pinref part="DISP" gate="G$1" pin="D6"/>
 <wire x1="-50.8" y1="-68.58" x2="-50.8" y2="-73.66" width="0.1524" layer="91"/>
 <label x="-50.8" y="-73.66" size="1.778" layer="95" rot="R270"/>
+</segment>
+<segment>
+<pinref part="IC2" gate="E" pin="O"/>
+<wire x1="167.64" y1="-104.14" x2="172.72" y2="-104.14" width="0.1524" layer="91"/>
+<label x="172.72" y="-104.14" size="1.778" layer="95"/>
 </segment>
 </net>
@@
 </segment>
 </net>
+<net name="N$7" class="0">
+<segment>
+<pinref part="IC2" gate="B" pin="O"/>
+<pinref part="IC2" gate="E" pin="I"/>
+<wire x1="142.24" y1="-104.14" x2="147.32" y2="-104.14" width="0.1524" layer="91"/>
+</segment>
+</net>
+<net name="N$8" class="0">
+<segment>
+<pinref part="SERIAL" gate="G$1" pin="7"/>
+<wire x1="129.54" y1="-76.2" x2="111.76" y2="-76.2" width="0.1524" layer="91"/>
+<wire x1="111.76" y1="-76.2" x2="111.76" y2="-104.14" width="0.1524" layer="91"/>
+<pinref part="IC2" gate="B" pin="I"/>
+<wire x1="111.76" y1="-104.14" x2="121.92" y2="-104.14" width="0.1524" layer="91"/>
+</segment>
+</net>

Commit message: Added SKAARHOJ_ID to a lot of PCBs...
Parts:
- C1: value 0.1uF -> 100nF
Changed lines of the file:
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@@
 <?xml version="1.0" encoding="utf-8"?>
 <!DOCTYPE eagle SYSTEM "eagle.dtd">
-<eagle version="7.1.0">
+<eagle version="7.7.0">
 <drawing>
 <settings>
@@
 <grid distance="0.1" unitdist="inch" unit="inch" style="lines" multiple="1" display="no" altdistance="0.01" altunitdist="inch" altunit="inch"/>
 <layers>
-<layer number="1" name="Top" color="4" fill="1" visible="no" active="no"/>
-<layer number="2" name="Route2" color="1" fill="3" visible="no" active="no"/>
-<layer number="3" name="Route3" color="4" fill="3" visible="no" active="no"/>
-<layer number="4" name="Route4" color="1" fill="4" visible="no" active="no"/>
-<layer number="5" name="Route5" color="4" fill="4" visible="no" active="no"/>
-<layer number="6" name="Route6" color="1" fill="8" visible="no" active="no"/>
-<layer number="7" name="Route7" color="4" fill="8" visible="no" active="no"/>
-<layer number="8" name="Route8" color="1" fill="2" visible="no" active="no"/>
-<layer number="9" name="Route9" color="4" fill="2" visible="no" active="no"/>
-<layer number="10" name="Route10" color="1" fill="7" visible="no" active="no"/>
-<layer number="11" name="Route11" color="4" fill="7" visible="no" active="no"/>
-<layer number="12" name="Route12" color="1" fill="5" visible="no" active="no"/>
-<layer number="13" name="Route13" color="4" fill="5" visible="no" active="no"/>
-<layer number="14" name="Route14" color="1" fill="6" visible="no" active="no"/>
-<layer number="15" name="Route15" color="4" fill="6" visible="no" active="no"/>
-<layer number="16" name="Bottom" color="1" fill="1" visible="no" active="no"/>
-<layer number="17" name="Pads" color="2" fill="1" visible="no" active="no"/>
-<layer number="18" name="Vias" color="2" fill="1" visible="no" active="no"/>
-<layer number="19" name="Unrouted" color="13" fill="1" visible="no" active="no"/>
-<layer number="20" name="Dimension" color="15" fill="1" visible="no" active="no"/>
-<layer number="21" name="tPlace" color="7" fill="1" visible="no" active="no"/>
-<layer number="22" name="bPlace" color="7" fill="1" visible="no" active="no"/>
-<layer number="23" name="tOrigins" color="15" fill="1" visible="no" active="no"/>
-<layer number="24" name="bOrigins" color="15" fill="1" visible="no" active="no"/>
-<layer number="25" name="tNames" color="7" fill="1" visible="no" active="no"/>
-<layer number="26" name="bNames" color="7" fill="1" visible="no" active="no"/>
-<layer number="27" name="tValues" color="7" fill="1" visible="no" active="no"/>
-<layer number="28" name="bValues" color="7" fill="1" visible="no" active="no"/>
+<layer number="1" name="Top" color="4" fill="1" visible="yes" active="no"/>
+<layer number="2" name="Route2" color="1" fill="3" visible="yes" active="no"/>
+<layer number="3" name="Route3" color="4" fill="3" visible="yes" active="no"/>
+<layer number="4" name="Route4" color="1" fill="4" visible="yes" active="no"/>
+<layer number="5" name="Route5" color="4" fill="4" visible="yes" active="no"/>
+<layer number="6" name="Route6" color="1" fill="8" visible="yes" active="no"/>
+<layer number="7" name="Route7" color="4" fill="8" visible="yes" active="no"/>
+<layer number="8" name="Route8" color="1" fill="2" visible="yes" active="no"/>
+<layer number="9" name="Route9" color="4" fill="2" visible="yes" active="no"/>
+<layer number="10" name="Route10" color="1" fill="7" visible="yes" active="no"/>
+<layer number="11" name="Route11" color="4" fill="7" visible="yes" active="no"/>
+<layer number="12" name="Route12" color="1" fill="5" visible="yes" active="no"/>
+<layer number="13" name="Route13" color="4" fill="5" visible="yes" active="no"/>
+<layer number="14" name="Route14" color="1" fill="6" visible="yes" active="no"/>
+<layer number="15" name="Route15" color="4" fill="6" visible="yes" active="no"/>
+<layer number="16" name="Bottom" color="1" fill="1" visible="yes" active="no"/>
+<layer number="17" name="Pads" color="2" fill="1" visible="yes" active="no"/>
+<layer number="18" name="Vias" color="2" fill="1" visible="yes" active="no"/>
+<layer number="19" name="Unrouted" color="13" fill="1" visible="yes" active="no"/>
+<layer number="20" name="Dimension" color="15" fill="1" visible="yes" active="no"/>
+<layer number="21" name="tPlace" color="7" fill="1" visible="yes" active="no"/>
+<layer number="22" name="bPlace" color="7" fill="1" visible="yes" active="no"/>
+<layer number="23" name="tOrigins" color="15" fill="1" visible="yes" active="no"/>
+<layer number="24" name="bOrigins" color="15" fill="1" visible="yes" active="no"/>
+<layer number="25" name="tNames" color="7" fill="1" visible="yes" active="no"/>
+<layer number="26" name="bNames" color="7" fill="1" visible="yes" active="no"/>
+<layer number="27" name="tValues" color="7" fill="1" visible="yes" active="no"/>
+<layer number="28" name="bValues" color="7" fill="1" visible="yes" active="no"/>
 <layer number="29" name="tStop" color="7" fill="3" visible="no" active="no"/>
 <layer number="30" name="bStop" color="7" fill="6" visible="no" active="no"/>
@@
 <layer number="35" name="tGlue" color="7" fill="4" visible="no" active="no"/>
 <layer number="36" name="bGlue" color="7" fill="5" visible="no" active="no"/>
-<layer number="37" name="tTest" color="7" fill="1" visible="no" active="no"/>
-<layer number="38" name="bTest" color="7" fill="1" visible="no" active="no"/>
+<layer number="37" name="tTest" color="7" fill="1" visible="yes" active="no"/>
+<layer number="38" name="bTest" color="7" fill="1" visible="yes" active="no"/>
 <layer number="39" name="tKeepout" color="4" fill="11" visible="no" active="no"/>
 <layer number="40" name="bKeepout" color="1" fill="11" visible="no" active="no"/>
@@
 <layer number="44" name="Drills" color="7" fill="1" visible="no" active="no"/>
 <layer number="45" name="Holes" color="7" fill="1" visible="no" active="no"/>
-<layer number="46" name="Milling" color="3" fill="1" visible="no" active="no"/>
-<layer number="47" name="Measures" color="7" fill="1" visible="no" active="no"/>
-<layer number="48" name="Document" color="7" fill="1" visible="no" active="no"/>
-<layer number="49" name="Reference" color="7" fill="1" visible="no" active="no"/>
-<layer number="50" name="dxf" color="7" fill="1" visible="no" active="no"/>
-<layer number="51" name="tDocu" color="7" fill="1" visible="no" active="no"/>
-<layer number="52" name="bDocu" color="7" fill="1" visible="no" active="no"/>
-<layer number="53" name="tGND_GNDA" color="7" fill="9" visible="no" active="no"/>
-<layer number="54" name="bGND_GNDA" color="1" fill="9" visible="no" active="no"/>
-<layer number="56" name="wert" color="7" fill="1" visible="no" active="no"/>
-<layer number="57" name="tCAD" color="7" fill="1" visible="no" active="no"/>
+<layer number="46" name="Milling" color="3" fill="1" visible="yes" active="no"/>
+<layer number="47" name="Measures" color="7" fill="1" visible="yes" active="no"/>
+<layer number="48" name="Document" color="7" fill="1" visible="yes" active="no"/>
+<layer number="49" name="Reference" color="7" fill="1" visible="yes" active="no"/>
+<layer number="50" name="dxf" color="7" fill="1" visible="yes" active="no"/>
+<layer number="51" name="tDocu" color="7" fill="1" visible="yes" active="no"/>
+<layer number="52" name="bDocu" color="7" fill="1" visible="yes" active="no"/>
+<layer number="53" name="tGND_GNDA" color="7" fill="9" visible="yes" active="no"/>
+<layer number="54" name="bGND_GNDA" color="1" fill="9" visible="yes" active="no"/>
+<layer number="56" name="wert" color="7" fill="1" visible="yes" active="no"/>
+<layer number="57" name="tCAD" color="7" fill="1" visible="yes" active="no"/>
 <layer number="91" name="Nets" color="2" fill="1" visible="yes" active="yes"/>
 <layer number="92" name="Busses" color="1" fill="1" visible="yes" active="yes"/>
@@
 <part name="U$6" library="SparkFun" deviceset="5V" device=""/>
 <part name="GND1" library="SparkFun" deviceset="GND" device=""/>
-<part name="C1" library="SparkFun" deviceset="CAP" device="0603-CAP" value="0.1uF"/>
+<part name="C1" library="SparkFun" deviceset="CAP" device="0603-CAP" value="100nF"/>
 <part name="U$2" library="SKAARHOJ" deviceset="GNDPAD" device="6MM" value="GNDPAD6MM"/>
 <part name="U$20" library="SKAARHOJ" deviceset="GNDPAD" device="6MM" value="GNDPAD6MM"/>
