File: PCBs/PCB-DISPLAYDOGM3/PCB-DISPLAYDOGM3.brd (EAGLE design)
At the start: 72 x 35 mm, 20 parts, among them IC2 74HC14D

Commit message: Added SKAARHOJ_ID to a lot of PCBs...
Parts:
- C1: value 0.1uF -> 100nF
Changed lines of the file:
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@@
 <?xml version="1.0" encoding="utf-8"?>
 <!DOCTYPE eagle SYSTEM "eagle.dtd">
-<eagle version="7.5.0">
+<eagle version="7.7.0">
 <drawing>
 <settings>
@@
 <element name="SERIAL" library="SKAARHOJ" package="M2X4SMALLER" value="M04X2M2X4SMALLER" x="68.5" y="19.2" smashed="yes" rot="MR180">
 <attribute name="VALUE" x="63.42" y="23.645" size="1.27" layer="28" rot="MR180"/>
+<attribute name="SKAARHOJ_ID" value="SK_2x4header" x="68.5" y="19.2" size="1.778" layer="28" rot="MR180" display="off"/>
 </element>
 <element name="U$19" library="SKAARHOJ" package="3BITADDR_SMALL" value="3BITADDRSMALL" x="15.7" y="26.5" rot="MR0"/>
-<element name="U$23" library="SKAARHOJ" package="TSSOP24" value="PCA9671" x="11.7" y="16.3" rot="MR270"/>
+<element name="U$23" library="SKAARHOJ" package="TSSOP24" value="PCA9671" x="11.7" y="16.3" rot="MR270">
+<attribute name="SKAARHOJ_ID" value="SK_PCA9671" x="11.7" y="16.3" size="1.778" layer="28" rot="MR270" display="off"/>
+</element>
 <element name="R2" library="SparkFun" package="0603-RES" value="10K" x="17.2" y="19.3" smashed="yes" rot="MR270">
 <attribute name="NAME" x="16.438" y="20.189" size="0.7112" layer="26" font="vector" rot="MR270"/>
 <attribute name="VALUE" x="18.343" y="20.316" size="0.4064" layer="28" font="vector" rot="MR270"/>
-</element>
-<element name="C1" library="SparkFun" package="0603-CAP" value="0.1uF" x="11.2" y="22.3" smashed="yes" rot="MR180">
+<attribute name="SKAARHOJ_ID" value="SK_10K" x="17.2" y="19.3" size="1.778" layer="28" rot="MR270" display="off"/>
+</element>
+<element name="C1" library="SparkFun" package="0603-CAP" value="100nF" x="11.2" y="22.3" smashed="yes" rot="MR180">
 <attribute name="NAME" x="10.311" y="21.538" size="0.7112" layer="26" font="vector" rot="MR180"/>
 <attribute name="VALUE" x="10.184" y="23.443" size="0.4064" layer="28" font="vector" rot="MR180"/>
+<attribute name="SKAARHOJ_ID" value="SK_100nF" x="11.2" y="22.3" size="1.778" layer="28" rot="MR180" display="off"/>
 </element>
 <element name="U$2" library="SKAARHOJ" package="3.2MMPAD6MM" value="GNDPAD6MM" x="3.5" y="31.5"/>
@@
 <element name="U$7" library="SKAARHOJ" package="3.2MMPAD6MM" value="GNDPAD6MM" x="68.5" y="3.5"/>
 <element name="U$21" library="SKAARHOJ" package="3.2MMPAD6MM" value="GNDPAD6MM" x="3.5" y="3.6"/>
-<element name="IC2" library="74xx-eu" package="SO14" value="74HC14D" x="55.2" y="17.8" rot="MR270"/>
+<element name="IC2" library="74xx-eu" package="SO14" value="74HC14D" x="55.2" y="17.8" rot="MR270">
+<attribute name="SKAARHOJ_ID" value="SK_74HCT14" x="55.2" y="17.8" size="1.778" layer="28" rot="MR270" display="off"/>
+</element>
 <element name="C18" library="SparkFun" package="0603-CAP" value="100nF" x="48.7" y="20.3" smashed="yes" rot="MR90">
 <attribute name="NAME" x="49.462" y="19.411" size="0.7112" layer="26" font="vector" rot="MR90"/>
 <attribute name="VALUE" x="47.557" y="19.284" size="0.4064" layer="28" font="vector" rot="MR90"/>
-</element>
-<element name="PC2" library="rcl" package="PANASONIC_D" value="100uF" x="26.4" y="17.5" rot="MR0"/>
+<attribute name="SKAARHOJ_ID" value="SK_100nF" x="48.7" y="20.3" size="1.778" layer="28" rot="MR90" display="off"/>
+</element>
+<element name="PC2" library="rcl" package="PANASONIC_D" value="100uF" x="26.4" y="17.5" rot="MR0">
+<attribute name="SKAARHOJ_ID" value="SK_100uF" x="26.4" y="17.5" size="1.778" layer="28" rot="MR0" display="off"/>
+</element>
 <element name="L4" library="SparkFun" package="0805" value="ILHB0805ER121V" x="69.6" y="9.7" smashed="yes" rot="MR270">
 <attribute name="NAME" x="68.7745" y="10.462" size="0.7112" layer="26" rot="MR270"/>
 <attribute name="VALUE" x="70.997" y="10.716" size="0.4064" layer="28" rot="MR270"/>
+<attribute name="SKAARHOJ_ID" value="SK_10uHBEAD" x="69.6" y="9.7" size="1.778" layer="28" rot="MR270" display="off"/>
 </element>
 <element name="C2" library="SparkFun" package="0805" value="22uF" x="66.8" y="7.9" smashed="yes" rot="MR0">
 <attribute name="NAME" x="67.562" y="8.7255" size="0.7112" layer="26" rot="MR0"/>
 <attribute name="VALUE" x="67.816" y="6.503" size="0.4064" layer="28" rot="MR0"/>
+<attribute name="SKAARHOJ_ID" value="SK_22uF" x="66.8" y="7.9" size="1.778" layer="28" rot="MR0" display="off"/>
 </element>
 <element name="C10" library="SparkFun" package="0603-CAP" value="100nF" x="66.7" y="9.8" smashed="yes" rot="MR0">
 <attribute name="NAME" x="67.589" y="10.562" size="0.7112" layer="26" font="vector" rot="MR0"/>
 <attribute name="VALUE" x="67.716" y="8.657" size="0.4064" layer="28" font="vector" rot="MR0"/>
+<attribute name="SKAARHOJ_ID" value="SK_100nF" x="66.7" y="9.8" size="1.778" layer="28" rot="MR0" display="off"/>
 </element>
 <element name="C12" library="SparkFun" package="0603-CAP" value="100nF" x="69.1" y="12.4" smashed="yes" rot="MR0">
 <attribute name="NAME" x="69.989" y="13.162" size="0.7112" layer="26" font="vector" rot="MR0"/>
 <attribute name="VALUE" x="70.116" y="11.257" size="0.4064" layer="28" font="vector" rot="MR0"/>
-</element>
-<element name="R1" library="SparkFun" package="0603-RES" value="?R" x="14" y="8" rot="MR90"/>
-<element name="R3" library="SparkFun" package="0603-RES" value="?R" x="60" y="8" rot="MR90"/>
-<element name="R4" library="SparkFun" package="0603-RES" value="?R" x="57" y="8" rot="MR90"/>
+<attribute name="SKAARHOJ_ID" value="SK_100nF" x="69.1" y="12.4" size="1.778" layer="28" rot="MR0" display="off"/>
+</element>
+<element name="R1" library="SparkFun" package="0603-RES" value="?R" x="14" y="8" rot="MR90">
+<attribute name="SKAARHOJ_ID" value="SK_33R" x="14" y="8" size="1.778" layer="28" rot="MR90" display="off"/>
+</element>
+<element name="R3" library="SparkFun" package="0603-RES" value="?R" x="60" y="8" rot="MR90">
+<attribute name="SKAARHOJ_ID" value="SK_33R" x="60" y="8" size="1.778" layer="28" rot="MR90" display="off"/>
+</element>
+<element name="R4" library="SparkFun" package="0603-RES" value="?R" x="57" y="8" rot="MR90">
+<attribute name="SKAARHOJ_ID" value="SK_33R" x="57" y="8" size="1.778" layer="28" rot="MR90" display="off"/>
+</element>
 </elements>
 <signals>
@@
 <contactref element="U$7" pad="P$1"/>
 <contactref element="U$21" pad="P$1"/>
-<contactref element="IC2" pad="7"/>
 <contactref element="C18" pad="2"/>
 <contactref element="PC2" pad="-"/>

Commit message: New resistor values for the RGB backlight (so balanced for white, less intense)
Parts:
- R1: value ?R -> 120R
- R3: value ?R -> 510R
- R4: value ?R -> 200R
Changed lines of the file:
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@@
 <attribute name="SKAARHOJ_ID" value="SK_100nF" x="69.1" y="12.4" size="1.778" layer="28" rot="MR0" display="off"/>
 </element>
-<element name="R1" library="SparkFun" package="0603-RES" value="?R" x="14" y="8" rot="MR90">
-<attribute name="SKAARHOJ_ID" value="SK_33R" x="14" y="8" size="1.778" layer="28" rot="MR90" display="off"/>
+<element name="R1" library="SparkFun" package="0603-RES" value="120R" x="14" y="8" rot="MR90">
+<attribute name="SKAARHOJ_ID" value="SK_120R" x="14" y="8" size="1.778" layer="28" rot="MR90" display="off"/>
 </element>
-<element name="R3" library="SparkFun" package="0603-RES" value="?R" x="60" y="8" rot="MR90">
-<attribute name="SKAARHOJ_ID" value="SK_33R" x="60" y="8" size="1.778" layer="28" rot="MR90" display="off"/>
+<element name="R3" library="SparkFun" package="0603-RES" value="510R" x="60" y="8" rot="MR90">
+<attribute name="SKAARHOJ_ID" value="SK_510R" x="60" y="8" size="1.778" layer="28" rot="MR90" display="off"/>
 </element>
-<element name="R4" library="SparkFun" package="0603-RES" value="?R" x="57" y="8" rot="MR90">
-<attribute name="SKAARHOJ_ID" value="SK_33R" x="57" y="8" size="1.778" layer="28" rot="MR90" display="off"/>
+<element name="R4" library="SparkFun" package="0603-RES" value="200R" x="57" y="8" rot="MR90">
+<attribute name="SKAARHOJ_ID" value="SK_200R" x="57" y="8" size="1.778" layer="28" rot="MR90" display="off"/>
 </element>
 </elements>

Commit message: d
Parts:
- R1: value 120R -> 120R/1%
- R3: value 510R -> 510R/1%
- R4: value 200R -> 200R/1%
Changed lines of the file:
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@@
 <attribute name="SKAARHOJ_ID" value="SK_100nF" x="69.1" y="12.4" size="1.778" layer="28" rot="MR0" display="off"/>
 </element>
-<element name="R1" library="SparkFun" package="0603-RES" value="120R" x="14" y="8" rot="MR90">
+<element name="R1" library="SparkFun" package="0603-RES" value="120R/1%" x="14" y="8" rot="MR90">
 <attribute name="SKAARHOJ_ID" value="SK_120R" x="14" y="8" size="1.778" layer="28" rot="MR90" display="off"/>
 </element>
-<element name="R3" library="SparkFun" package="0603-RES" value="510R" x="60" y="8" rot="MR90">
+<element name="R3" library="SparkFun" package="0603-RES" value="510R/1%" x="60" y="8" rot="MR90">
 <attribute name="SKAARHOJ_ID" value="SK_510R" x="60" y="8" size="1.778" layer="28" rot="MR90" display="off"/>
 </element>
-<element name="R4" library="SparkFun" package="0603-RES" value="200R" x="57" y="8" rot="MR90">
+<element name="R4" library="SparkFun" package="0603-RES" value="200R/1%" x="57" y="8" rot="MR90">
 <attribute name="SKAARHOJ_ID" value="SK_200R" x="57" y="8" size="1.778" layer="28" rot="MR90" display="off"/>
 </element>
