File: PCBs/PCB-JOY-4AXIS/PCB-JOY-4AXIS_adaptorHirose.brd (EAGLE design)
At the start: 50 x 50 mm, 5 parts

Commit message: 4AXISHirose
Parts:
- moved U$2 1.00 mm to (10.0, 31.0)
Connections:
- new net N$1: U$2.2, U$5.LR_V, U$5.ROT_V, U$5.UD_V
- new net N$2: U$2.4, U$5.LR_C
- new net N$3: U$2.6, U$5.UD_C
- new net N$4: U$2.8, U$5.ROT_C
- new net N$5: JP1.1, U$2.9
- net GND: now also JP1.2, U$2.1, U$2.10, U$5.LR_COM, U$5.ROT_COM, U$5.UD_COM
Routing:
- net GND: track 0.00 -> 106.5 mm, vias 0 -> 1
- net N$1: track 0.00 -> 58.4 mm, vias 0 -> 1
- net N$2: track 0.00 -> 48.9 mm
- net N$5: track 0.00 -> 24.7 mm
- net N$4: track 0.00 -> 20.0 mm, vias 0 -> 2
- net N$3: track 0.00 -> 8.02 mm
- added copper zone on layer 1, net GND
- added copper zone on layer 16, net GND
Other:
- outline, holes or cut-outs redrawn
Changed lines of the file:
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@@
 <wire x1="9" y1="25" x2="9" y2="9" width="0" layer="20"/>
 <wire x1="9" y1="9" x2="50" y2="9" width="0" layer="20"/>
-<wire x1="9" y1="37" x2="11" y2="37" width="0" layer="20"/>
-<wire x1="11" y1="37" x2="11" y2="25" width="0" layer="20"/>
-<wire x1="11" y1="25" x2="9" y2="25" width="0" layer="20"/>
+<wire x1="9" y1="37" x2="10" y2="37" width="0" layer="20"/>
+<wire x1="10" y1="37" x2="10" y2="25" width="0" layer="20"/>
+<wire x1="10" y1="25" x2="9" y2="25" width="0" layer="20"/>
 </plain>
 <attributes>
@@
 <element name="U$1" library="SKAARHOJ" package="3.2MMPAD6MM" value="GNDPAD6MM" x="3.5" y="46.5"/>
 <element name="U$6" library="SKAARHOJ" package="3.2MMPAD6MM" value="GNDPAD6MM" x="46.5" y="3.5"/>
-<element name="U$2" library="SKAARHOJ" package="2X6HIROSE_DF11-12DS-2DSA" value="HIROSE-DF11-12DS-2DSA" x="11" y="31"/>
+<element name="U$2" library="SKAARHOJ" package="2X6HIROSE_DF11-12DS-2DSA" value="HIROSE-DF11-12DS-2DSA" x="10" y="31"/>
 </elements>
 <signals>
@@
 <contactref element="U$1" pad="P$1"/>
 <contactref element="U$6" pad="P$1"/>
-<wire x1="46.5" y1="3.5" x2="3.5" y2="46.5" width="0" layer="19" extent="1-1"/>
+<contactref element="JP1" pad="2"/>
+<contactref element="U$5" pad="LR_COM"/>
+<contactref element="U$5" pad="UD_COM"/>
+<contactref element="U$5" pad="ROT_COM"/>
+<contactref element="U$2" pad="1"/>
+<contactref element="U$2" pad="10"/>
+<wire x1="43.9928" y1="1.016" x2="36.068" y2="1.016" width="0.3048" layer="1"/>
+<wire x1="46.4312" y1="3.4544" x2="43.9928" y2="1.016" width="0.3048" layer="1"/>
+<wire x1="36.068" y1="1.016" x2="36" y2="1" width="0.3048" layer="1"/>
+<wire x1="46.4312" y1="3.4544" x2="46.5" y2="3.5" width="0.3048" layer="1"/>
+<wire x1="7.0104" y1="23.9776" x2="8.9408" y2="25.908" width="0.3048" layer="16"/>
+<wire x1="7.0104" y1="14.6304" x2="7.0104" y2="23.9776" width="0.3048" layer="1"/>
+<wire x1="8.9408" y1="25.908" x2="9" y2="26" width="0.3048" layer="16"/>
+<wire x1="7.0104" y1="14.6304" x2="7" y2="14.54" width="0.3048" layer="1"/>
+<wire x1="2.54" y1="18.9992" x2="2.032" y2="18.9992" width="0.3048" layer="16"/>
+<wire x1="2.032" y1="18.9992" x2="1.016" y2="18.9992" width="0.3048" layer="16"/>
+<wire x1="6.9088" y1="14.6304" x2="2.54" y2="18.9992" width="0.3048" layer="16"/>
+<wire x1="1.016" y1="18.9992" x2="1" y2="19" width="0.3048" layer="16"/>
+<wire x1="6.9088" y1="14.6304" x2="7" y2="14.54" width="0.3048" layer="16"/>
+<wire x1="2.9464" y1="34.036" x2="8.9408" y2="34.036" width="0.3048" layer="1"/>
+<wire x1="1.016" y1="35.9664" x2="2.9464" y2="34.036" width="0.3048" layer="1"/>
+<wire x1="8.9408" y1="34.036" x2="9" y2="34" width="0.3048" layer="1"/>
+<wire x1="1.016" y1="35.9664" x2="1" y2="36" width="0.3048" layer="1"/>
+<wire x1="1.1176" y1="44.0944" x2="1.1176" y2="36.068" width="0.3048" layer="1"/>
+<wire x1="3.4544" y1="46.4312" x2="1.1176" y2="44.0944" width="0.3048" layer="1"/>
+<wire x1="1.1176" y1="36.068" x2="1" y2="36" width="0.3048" layer="1"/>
+<wire x1="3.4544" y1="46.4312" x2="3.5" y2="46.5" width="0.3048" layer="1"/>
+<wire x1="2.032" y1="34.9504" x2="2.032" y2="18.9992" width="0.3048" layer="16"/>
+<wire x1="1.016" y1="35.9664" x2="2.032" y2="34.9504" width="0.3048" layer="16"/>
+<wire x1="1.016" y1="35.9664" x2="1" y2="36" width="0.3048" layer="16"/>
+<wire x1="31.8008" y1="1.016" x2="35.8648" y2="1.016" width="0.3048" layer="1"/>
+<wire x1="24.2824" y1="8.5344" x2="31.8008" y2="1.016" width="0.3048" layer="1"/>
+<wire x1="8.8392" y1="8.5344" x2="24.2824" y2="8.5344" width="0.3048" layer="1"/>
+<wire x1="8.3312" y1="9.0424" x2="8.8392" y2="8.5344" width="0.3048" layer="1"/>
+<wire x1="8.3312" y1="13.1064" x2="8.3312" y2="9.0424" width="0.3048" layer="1"/>
+<wire x1="7.0104" y1="14.4272" x2="8.3312" y2="13.1064" width="0.3048" layer="1"/>
+<wire x1="35.8648" y1="1.016" x2="36" y2="1" width="0.3048" layer="1"/>
+<wire x1="7.0104" y1="14.4272" x2="7" y2="14.54" width="0.3048" layer="1"/>
+<via x="7.0104" y="23.9776" extent="1-16" drill="0.6096"/>
+<polygon width="0.4064" layer="16">
+<vertex x="0" y="0"/>
+<vertex x="50" y="0"/>
+<vertex x="50" y="50"/>
+<vertex x="0" y="50"/>
+</polygon>
+<polygon width="0.4064" layer="1">
+<vertex x="0" y="0"/>
+<vertex x="50" y="0"/>
+<vertex x="50" y="50"/>
+<vertex x="0" y="50"/>
+</polygon>
+</signal>
+<signal name="N$1">
+<contactref element="U$5" pad="ROT_V"/>
+<contactref element="U$5" pad="UD_V"/>
+<contactref element="U$5" pad="LR_V"/>
+<contactref element="U$2" pad="2"/>
+<wire x1="7.8232" y1="25.908" x2="8.9408" y2="25.908" width="0.2032" layer="1"/>
+<wire x1="5.2832" y1="23.368" x2="7.8232" y2="25.908" width="0.2032" layer="1"/>
+<wire x1="5.2832" y1="16.3576" x2="5.2832" y2="23.368" width="0.2032" layer="1"/>
+<wire x1="4.6736" y1="15.748" x2="5.2832" y2="16.3576" width="0.2032" layer="1"/>
+<wire x1="3.7592" y1="15.748" x2="4.6736" y2="15.748" width="0.2032" layer="16"/>
+<wire x1="1.016" y1="13.0048" x2="2.5908" y2="14.5796" width="0.2032" layer="16"/>
+<wire x1="2.5908" y1="14.5796" x2="3.7592" y2="15.748" width="0.2032" layer="16"/>
+<wire x1="8.9408" y1="25.908" x2="9" y2="26" width="0.2032" layer="1"/>
+<wire x1="1.016" y1="13.0048" x2="1" y2="13" width="0.2032" layer="16"/>
+<wire x1="16.1544" y1="1.016" x2="23.9776" y2="1.016" width="0.2032" layer="16"/>
+<wire x1="2.5908" y1="14.5796" x2="16.1544" y2="1.016" width="0.2032" layer="16"/>
+<wire x1="23.9776" y1="1.016" x2="24" y2="1" width="0.2032" layer="16"/>
+<wire x1="1.016" y1="22.5552" x2="1.016" y2="23.9776" width="0.2032" layer="1"/>
+<wire x1="4.4704" y1="19.1008" x2="1.016" y2="22.5552" width="0.2032" layer="1"/>
+<wire x1="4.4704" y1="17.1704" x2="4.4704" y2="19.1008" width="0.2032" layer="1"/>
+<wire x1="1.016" y1="13.716" x2="4.4704" y2="17.1704" width="0.2032" layer="1"/>
+<wire x1="1.016" y1="13.0048" x2="1.016" y2="13.716" width="0.2032" layer="1"/>
+<wire x1="1.016" y1="23.9776" x2="1" y2="24" width="0.2032" layer="1"/>
+<wire x1="1.016" y1="13.0048" x2="1" y2="13" width="0.2032" layer="1"/>
+<via x="4.6736" y="15.748" extent="1-16" drill="0.4064"/>
+</signal>
+<signal name="N$2">
+<contactref element="U$5" pad="LR_C"/>
+<contactref element="U$2" pad="4"/>
+<wire x1="7.8232" y1="27.94" x2="8.9408" y2="27.94" width="0.2032" layer="1"/>
+<wire x1="4.8768" y1="24.9936" x2="7.8232" y2="27.94" width="0.2032" layer="1"/>
+<wire x1="4.8768" y1="16.9672" x2="4.8768" y2="24.9936" width="0.2032" layer="1"/>
+<wire x1="3.9624" y1="16.0528" x2="4.8768" y2="16.9672" width="0.2032" layer="1"/>
+<wire x1="3.9624" y1="12.7" x2="3.9624" y2="16.0528" width="0.2032" layer="1"/>
+<wire x1="14.6304" y1="2.032" x2="3.9624" y2="12.7" width="0.2032" layer="1"/>
+<wire x1="28.956" y1="2.032" x2="14.6304" y2="2.032" width="0.2032" layer="1"/>
+<wire x1="29.972" y1="1.016" x2="28.956" y2="2.032" width="0.2032" layer="1"/>
+<wire x1="8.9408" y1="27.94" x2="9" y2="28" width="0.2032" layer="1"/>
+<wire x1="29.972" y1="1.016" x2="30" y2="1" width="0.2032" layer="1"/>
+</signal>
+<signal name="N$3">
+<contactref element="U$5" pad="UD_C"/>
+<contactref element="U$2" pad="6"/>
+<wire x1="1.016" y1="29.972" x2="8.9408" y2="29.972" width="0.2032" layer="1"/>
+<wire x1="8.9408" y1="29.972" x2="9" y2="30" width="0.2032" layer="1"/>
+<wire x1="1.016" y1="29.972" x2="1" y2="30" width="0.2032" layer="1"/>
+</signal>
+<signal name="N$4">
+<contactref element="U$5" pad="ROT_C"/>
+<contactref element="U$2" pad="8"/>
+<wire x1="7.8232" y1="31.9024" x2="8.9408" y2="31.9024" width="0.2032" layer="1"/>
+<wire x1="6.604" y1="30.6832" x2="7.8232" y2="31.9024" width="0.2032" layer="1"/>
+<wire x1="6.604" y1="25.2984" x2="6.604" y2="30.6832" width="0.2032" layer="16"/>
+<wire x1="3.7592" y1="22.4536" x2="6.604" y2="25.2984" width="0.2032" layer="16"/>
+<wire x1="3.7592" y1="18.796" x2="3.7592" y2="22.4536" width="0.2032" layer="16"/>
+<wire x1="1.016" y1="16.0528" x2="3.7592" y2="18.796" width="0.2032" layer="1"/>
+<wire x1="8.9408" y1="31.9024" x2="9" y2="32" width="0.2032" layer="1"/>
+<wire x1="1.016" y1="16.0528" x2="1" y2="16" width="0.2032" layer="1"/>
+<via x="6.604" y="30.6832" extent="1-16" drill="0.4064"/>
+<via x="3.7592" y="18.796" extent="1-16" drill="0.4064"/>
+</signal>
+<signal name="N$5">
+<contactref element="JP1" pad="1"/>
+<contactref element="U$2" pad="9"/>
+<wire x1="8.0264" y1="33.02" x2="8.9408" y2="33.9344" width="0.2032" layer="16"/>
+<wire x1="7.9248" y1="33.02" x2="8.0264" y2="33.02" width="0.2032" layer="16"/>
+<wire x1="7.3152" y1="32.4104" x2="7.9248" y2="33.02" width="0.2032" layer="16"/>
+<wire x1="7.3152" y1="25.4" x2="7.3152" y2="32.4104" width="0.2032" layer="16"/>
+<wire x1="6.1976" y1="24.2824" x2="7.3152" y2="25.4" width="0.2032" layer="16"/>
+<wire x1="6.1976" y1="17.1704" x2="6.1976" y2="24.2824" width="0.2032" layer="16"/>
+<wire x1="8.3312" y1="15.0368" x2="6.1976" y2="17.1704" width="0.2032" layer="16"/>
+<wire x1="8.3312" y1="13.4112" x2="8.3312" y2="15.0368" width="0.2032" layer="16"/>
+<wire x1="7.0104" y1="12.0904" x2="8.3312" y2="13.4112" width="0.2032" layer="16"/>
+<wire x1="8.9408" y1="33.9344" x2="9" y2="34" width="0.2032" layer="16"/>
+<wire x1="7.0104" y1="12.0904" x2="7" y2="12" width="0.2032" layer="16"/>
 </signal>
 </signals>
